File: alphax_4ch.kicad_sch (KiCad schematic)
At the start: 245 parts, among them J1 USB_B_Mini, J2 Cortex_Debug, J3 Conn_01x01, J4 Conn_01x01, J5 Conn_01x01, J6 Conn_01x01, J7 Conn_01x01, J8 Conn_01x01, M1 Module-power12-0.2, M2 Module-power5-0.2, M3 Module-vr-discrete-0.1, M4 Module-ign8-0.2, M5 Module-input-0.1, M6 Module-mcu144-0.6, M7 Module-can-0.1, M8 Module-vr-discrete-0.1, M9 Module-knock-0.1, P1 33311-24AW-2, P2 33311-24AW-2, Q1 AO3400A, Q10 AO3400A, Q11 AO3400A, Q12 AO3400A, Q13 AO3401A, Q14 AO3401A, Q15 AO3400A, Q16 AO3401A, Q17 AO3401A, Q18 AO3401A, Q19 AO3400A, Q2 AO3400A, Q20 AO3400A, Q21 AO3400A, Q22 VND14NV04-E, Q23 VND14NV04-E, Q24 AO3400A, Q25 AO3400A, Q26 VND14NV04-E, Q27 AO3400A, Q28 VND14NV04-E, Q29 VND14NV04-E, Q3 AO3401A, Q30 VND14NV04-E, Q31 AO3401A, Q32 AO3401A, Q33 AO3400A, Q34 AO3400A, Q35 AO3400A, Q36 AO3400A, Q4 AO3401A, Q5 AO3401A, Q6 VND14NV04-E, Q7 VND14NV04-E, Q8 VND14NV04-E, Q9 VND14NV04-E, U1 TLS115, U2 74HC2G17GW, U3 MPXH6400A, U4 JDY-33, U5 74HC2G17GW, U6 TLE9201SG, U7 SN74LVC1G06DBVR

Commit message: https://github.com/rusefi/alphax-4chan/issues/34
Parts:
- added R94, R95: 510k, hellen-one-common:R0603, symbol hellen-one-common:Res
Connections:
- net GND: now also R94.2, R95.2
- net GNDA: no longer M5.J10 (PULL_AUX1), M5.J9 (PULL_AUX2)
- net IN_PPS2: now also R95.1
- net IN_TPS2: now also R94.1
- no-connect marks 74 -> 76
Changed lines of the file:
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@@
   (title_block
     (title "AlphaECU 4chan powered by rusEFI")
-    (date "2022-06-10")
+    (date "2022-06-13")
     (rev "C")
     (company "rusEFI")
@@
   (no_connect (at 461.01 276.86))
   (no_connect (at 241.3 187.96))
+  (no_connect (at 461.01 261.62))
   (no_connect (at 349.25 219.71))
   (no_connect (at 233.68 46.99))
@@
   (no_connect (at 361.95 294.64))
   (no_connect (at 317.5 114.3))
+  (no_connect (at 461.01 259.08))
   (no_connect (at 402.59 325.12))
   (no_connect (at 457.2 52.07))
@@
     (stroke (width 0) (type default) (color 0 0 0 0))
   )
+  (wire (pts (xy 314.96 321.31) (xy 325.12 321.31))
+    (stroke (width 0) (type default) (color 0 0 0 0))
+  )
   (bus (pts (xy 184.15 208.28) (xy 184.15 227.33))
     (stroke (width 0.3048) (type solid) (color 255 255 0 1))
@@
     (stroke (width 0) (type default) (color 0 0 0 0))
   )
+  (wire (pts (xy 314.96 325.12) (xy 325.12 325.12))
+    (stroke (width 0) (type default) (color 0 0 0 0))
+  )
   (wire (pts (xy 132.08 132.08) (xy 193.04 132.08))
     (stroke (width 0) (type default) (color 0 0 0 0))
@@
     (effects (font (size 1.27 1.27)) (justify left bottom))
   )
+  (label "IN_TPS2" (at 316.23 321.31 0)
+    (effects (font (size 1.27 1.27)) (justify left bottom))
+  )
   (label "NOS" (at 321.31 72.39 0)
     (effects (font (size 1.27 1.27)) (justify left bottom))
@@
     (effects (font (size 1.27 1.27)) (justify right bottom))
   )
+  (label "IN_PPS2" (at 316.23 325.12 0)
+    (effects (font (size 1.27 1.27)) (justify left bottom))
+  )
   (label "OUT_VVT2" (at 231.14 132.08 0)
     (effects (font (size 1.27 1.27)) (justify left bottom))
@@
     (pin "1")
   )
-  (symbol (lib_id "power:GNDA") (at 461.01 259.08 90) (unit 1)
-    (in_bom yes) (on_board yes)
-    (property "Reference" "#PWR075" (id 0) (at 467.36 259.08 0)
-      (effects (font (size 1.27 1.27)) hide)
-    )
-    (property "Value" "GNDA" (id 1) (at 466.448 259.2439 90))
-    (property "Footprint" "" (id 2) (at 461.01 259.08 0)
-      (effects (font (size 1.27 1.27)) hide)
-    )
-    (property "Datasheet" "" (id 3) (at 461.01 259.08 0)
-      (effects (font (size 1.27 1.27)) hide)
-    )
-    (pin "1")
-  )
   (symbol (lib_id "hellen-one-common:Jumper-Pad-Pad") (at 127 85.09 0) (mirror y) (unit 1)
     (in_bom yes) (on_board yes)
@@
     (pin "3")
   )
+  (symbol (lib_id "power:GND") (at 335.28 325.12 90) (unit 1)
+    (in_bom yes) (on_board yes)
+    (property "Reference" "#PWR0131" (id 0) (at 341.63 325.12 0)
+      (effects (font (size 1.27 1.27)) hide)
+    )
+    (property "Value" "GND" (id 1) (at 339.2234 325.0692 0))
+    (property "Footprint" "" (id 2) (at 335.28 325.12 0)
+      (effects (font (size 1.27 1.27)) hide)
+    )
+    (property "Datasheet" "" (id 3) (at 335.28 325.12 0)
+      (effects (font (size 1.27 1.27)) hide)
+    )
+    (pin "1")
+  )
   (symbol (lib_id "hellen-one-common:Fuse-Pad-Pad") (at 127 115.57 0) (unit 1)
     (in_bom yes) (on_board yes)
@@
     (pin "2")
   )
+  (symbol (lib_id "hellen-one-common:Res") (at 325.12 321.31 0) (mirror x) (unit 1)
+    (in_bom yes) (on_board yes)
+    (property "Reference" "R94" (id 0) (at 330.2 318.77 0))
+    (property "Value" "510k" (id 1) (at 330.2 321.31 0))
+    (property "Footprint" "hellen-one-common:R0603" (id 2) (at 328.93 317.5 0)
+      (effects (font (size 1.27 1.27)) hide)
+    )
+    (property "Datasheet" "" (id 3) (at 325.12 321.31 0)
+      (effects (font (size 1.27 1.27)) hide)
+    )
+    (property "LCSC" "C23192" (id 4) (at 325.12 321.31 0)
+      (effects (font (size 1.27 1.27)) hide)
+    )
+    (pin "1")
+    (pin "2")
+  )
   (symbol (lib_id "hellen-one-common:Jumper-Pad-Pad") (at 127 172.72 0) (mirror y) (unit 1)
     (in_bom yes) (on_board yes)
@@
     (pin "2")
   )
+  (symbol (lib_id "hellen-one-common:Res") (at 325.12 325.12 0) (mirror x) (unit 1)
+    (in_bom yes) (on_board yes)
+    (property "Reference" "R95" (id 0) (at 330.2 327.66 0))
+    (property "Value" "510k" (id 1) (at 330.2 325.12 0))
+    (property "Footprint" "hellen-one-common:R0603" (id 2) (at 328.93 321.31 0)
+      (effects (font (size 1.27 1.27)) hide)
+    )
+    (property "Datasheet" "" (id 3) (at 325.12 325.12 0)
+      (effects (font (size 1.27 1.27)) hide)
+    )
+    (property "LCSC" "C23192" (id 4) (at 325.12 325.12 0)
+      (effects (font (size 1.27 1.27)) hide)
+    )
+    (pin "1")
+    (pin "2")
+  )
   (symbol (lib_id "power:+5V") (at 88.9 250.19 0) (unit 1)
     (in_bom yes) (on_board yes)
@@
     (pin "1")
   )
+  (symbol (lib_id "power:GND") (at 335.28 321.31 90) (unit 1)
+    (in_bom yes) (on_board yes)
+    (property "Reference" "#PWR0104" (id 0) (at 341.63 321.31 0)
+      (effects (font (size 1.27 1.27)) hide)
+    )
+    (property "Value" "GND" (id 1) (at 339.2234 321.2592 0))
+    (property "Footprint" "" (id 2) (at 335.28 321.31 0)
+      (effects (font (size 1.27 1.27)) hide)
+    )
+    (property "Datasheet" "" (id 3) (at 335.28 321.31 0)
+      (effects (font (size 1.27 1.27)) hide)
+    )
+    (pin "1")
+  )
   (symbol (lib_id "hellen-one-common:MOSFET-P") (at 223.52 279.4 0) (mirror x) (unit 1)
     (in_bom yes) (on_board yes)
@@
     (pin "2")
   )
-  (symbol (lib_id "power:GNDA") (at 461.01 261.62 90) (unit 1)
-    (in_bom yes) (on_board yes)
-    (property "Reference" "#PWR076" (id 0) (at 467.36 261.62 0)
-      (effects (font (size 1.27 1.27)) hide)
-    )
-    (property "Value" "GNDA" (id 1) (at 466.448 261.7839 90))
-    (property "Footprint" "" (id 2) (at 461.01 261.62 0)
-      (effects (font (size 1.27 1.27)) hide)
-    )
-    (property "Datasheet" "" (id 3) (at 461.01 261.62 0)
-      (effects (font (size 1.27 1.27)) hide)
-    )
-    (pin "1")
-  )
   (symbol (lib_id "hellen-one-common:Res_Array_4") (at 219.71 335.28 0) (unit 1)
     (in_bom yes) (on_board yes)
@@
       (reference "#PWR074") (unit 1) (value "GNDA") (footprint "")
     )
-    (path "/236fad3a-f0b0-4b66-8d87-b2c1e224be21"
-      (reference "#PWR075") (unit 1) (value "GNDA") (footprint "")
-    )
-    (path "/f8285b65-02a7-4092-88f9-49a6d6cb2309"
-      (reference "#PWR076") (unit 1) (value "GNDA") (footprint "")
-    )
     (path "/493d0df1-7663-448c-9f99-931744972c8b"
       (reference "#PWR077") (unit 1) (value "+5VA") (footprint "")
@@
       (reference "#PWR0103") (unit 1) (value "+5V") (footprint "")
     )
+    (path "/f40bafb5-64be-421f-89b6-b9e1037282e1"
+      (reference "#PWR0104") (unit 1) (value "GND") (footprint "")
+    )
     (path "/41489dcd-290f-47ff-9a59-909b0e450dc0"
       (reference "#PWR0105") (unit 1) (value "GND") (footprint "")
@@
       (reference "#PWR0130") (unit 1) (value "GND") (footprint "")
     )
+    (path "/8c3dc30c-2bf8-4ac4-9e34-5a25bed02740"
+      (reference "#PWR0131") (unit 1) (value "GND") (footprint "")
+    )
     (path "/ee8c4410-d8e1-435a-8bf6-9b69d94306ef"
       (reference "#PWR0132") (unit 1) (value "+5VAS") (footprint "")
@@
       (reference "R93") (unit 1) (value "4.7k") (footprint "hellen-one-common:R0603")
     )
+    (path "/cf78c488-1611-40a0-85fa-15bfae75637e"
+      (reference "R94") (unit 1) (value "510k") (footprint "hellen-one-common:R0603")
+    )
+    (path "/dede5982-788e-4422-a3af-a7f72e3578e0"
+      (reference "R95") (unit 1) (value "510k") (footprint "hellen-one-common:R0603")
+    )
     (path "/f5cf27f5-0f5a-41ca-bd1a-78dcac84a3d5"
