File: alphax_4ch.kicad_sch (KiCad schematic)
At the start: 245 parts, among them J1 USB_B_Mini, J10 Conn_01x01, J11 Conn_01x01, J2 Cortex_Debug, J3 Conn_01x01, J4 Conn_01x01, J5 Conn_01x01, J6 Conn_01x01, J7 Conn_01x01, J8 Conn_01x01, J9 Micro_SD_Card, M1 Module-power12-0.2, M2 Module-power5-0.2, M3 Module-vr-discrete-0.4, M4 Module-ign8-0.2, M5 Module-input-0.1, M6 Module-mcu144-0.6, M7 Module-can-0.1, M8 Module-vr-discrete-0.4, M9 Module-knock-0.2, P1 33311-24AW-2, P2 33311-24AW-2, Q1 AO3400A, Q10 AO3400A, Q11 AO3400A, Q12 AO3400A, Q13 AO3401A, Q14 AO3401A, Q15 AO3400A, Q16 AO3401A, Q17 AO3401A, Q18 AO3401A, Q19 AO3400A, Q2 AO3400A, Q20 AO3400A, Q21 AO3400A, Q22 VND14NV04-E, Q23 VND14NV04-E, Q24 AO3400A, Q25 AO3400A, Q26 VND14NV04-E, Q27 AO3400A, Q28 VND14NV04-E, Q29 VND14NV04-E, Q3 AO3401A, Q30 VND14NV04-E, Q31 AO3401A, Q32 AO3401A, Q33 AO3400A, Q34 AO3400A, Q35 AO3400A, Q36 AO3400A, Q4 AO3401A, Q5 AO3401A, Q6 VND14NV04-E, Q7 VND14NV04-E, Q8 VND14NV04-E, Q9 VND14NV04-E, U1 TLS115, U2 74HC2G17GW, U3 MPXH6400A, U4 JDY-33, U5 74HC2G17GW, U6 TLE9201SG, U7 SN74LVC1G06DBVR

Commit message: Upd PCB
Connections:
- now unconnected: U3.1, U3.5, U3.6, U3.7, U3.8
- no-connect marks 69 -> 74
Changed lines of the file:
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@@
   (title_block
     (title "AlphaECU 4chan powered by rusEFI")
-    (date "2022-09-05")
+    (date "2023-02-02")
     (rev "F")
     (company "rusEFI")
     (comment 7 "http://rusefi.com/s/alphax4ch")
   )
-  (junction (at 415.29 219.71) (diameter 0) (color 0 0 0 0)
-  )
   (junction (at 355.6 278.13) (diameter 0) (color 0 0 0 0)
   )
@@
   (junction (at 270.51 340.36) (diameter 0) (color 0 0 0 0)
   )
-  (junction (at 415.29 222.25) (diameter 0) (color 0 0 0 0)
-  )
-  (junction (at 415.29 224.79) (diameter 0) (color 0 0 0 0)
-  )
   (junction (at 25.4 351.79) (diameter 0) (color 0 0 0 0)
   )
@@
   (no_connect (at 233.68 41.91))
   (no_connect (at 457.2 69.85))
+  (no_connect (at 415.29 219.71))
   (no_connect (at 457.2 100.33))
   (no_connect (at 459.74 171.45))
   (no_connect (at 415.29 264.16))
+  (no_connect (at 415.29 217.17))
   (no_connect (at 349.25 229.87))
   (no_connect (at 457.2 39.37))
@@
   (no_connect (at 269.24 401.32))
   (no_connect (at 457.2 74.93))
+  (no_connect (at 415.29 222.25))
   (no_connect (at 571.5 361.95))
   (no_connect (at 457.2 72.39))
   (no_connect (at 311.15 237.49))
+  (no_connect (at 415.29 224.79))
   (no_connect (at 523.24 227.33))
   (no_connect (at 416.56 44.45))
@@
   (no_connect (at 457.2 36.83))
   (no_connect (at 85.09 215.9))
+  (no_connect (at 440.69 224.79))
   (no_connect (at 416.56 46.99))
   (no_connect (at 311.15 219.71))
@@
     (stroke (width 0) (type default) (color 0 0 0 0))
   )
-  (wire (pts (xy 440.69 224.79) (xy 440.69 227.33))
-    (stroke (width 0) (type default) (color 0 0 0 0))
-  )
   (wire (pts (xy 337.82 80.01) (xy 337.82 99.06))
     (stroke (width 0) (type default) (color 0 0 0 0))
@@
     (stroke (width 0) (type default) (color 0 0 0 0))
   )
-  (wire (pts (xy 415.29 217.17) (xy 415.29 219.71))
-    (stroke (width 0) (type default) (color 0 0 0 0))
-  )
   (wire (pts (xy 257.81 138.43) (xy 257.81 142.24))
     (stroke (width 0) (type default) (color 0 0 0 0))
@@
     (stroke (width 0) (type default) (color 0 0 0 0))
   )
-  (wire (pts (xy 415.29 227.33) (xy 440.69 227.33))
-    (stroke (width 0) (type default) (color 0 0 0 0))
-  )
   (wire (pts (xy 113.03 350.52) (xy 115.57 350.52))
     (stroke (width 0) (type solid) (color 0 0 0 0))
@@
     (stroke (width 0.3048) (type solid) (color 132 132 0 1))
   )
-  (wire (pts (xy 415.29 227.33) (xy 415.29 224.79))
-    (stroke (width 0) (type default) (color 0 0 0 0))
-  )
   (wire (pts (xy 219.71 339.09) (xy 232.41 339.09))
     (stroke (width 0) (type default) (color 0 0 0 0))
@@
     (stroke (width 0) (type solid) (color 0 0 0 0))
   )
-  (wire (pts (xy 415.29 219.71) (xy 415.29 222.25))
-    (stroke (width 0) (type default) (color 0 0 0 0))
-  )
   (wire (pts (xy 132.08 124.46) (xy 151.13 124.46))
     (stroke (width 0) (type default) (color 0 0 0 0))
@@
     (stroke (width 0) (type solid) (color 0 0 0 0))
   )
-  (wire (pts (xy 415.29 222.25) (xy 415.29 224.79))
-    (stroke (width 0) (type default) (color 0 0 0 0))
-  )
   (wire (pts (xy 381 110.49) (xy 416.56 110.49))

Commit message: #95
Connections:
- net at D44.1 (A): now also D38.1 (K); no longer D38.2 (A)
- net at D9.1 (A): now also D1.1 (K); no longer D1.2 (A)
- net at R50.5: now also D38.2 (A); no longer D38.1 (K)
- net at R50.7, R50.8: now also D1.2 (A); no longer D1.1 (K)
Changed lines of the file:
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@@
     (pin "3")
   )
-  (symbol (lib_id "hellen-one-common:1N4148WS") (at 123.19 350.52 0) (mirror y) (unit 1)
+  (symbol (lib_id "hellen-one-common:1N4148WS") (at 120.65 350.52 0) (mirror x) (unit 1)
     (in_bom yes) (on_board yes)
     (property "Reference" "D38" (id 0) (at 115.57 351.79 0))
-    (property "Value" "1N4148WS" (id 1) (at 119.38 354.33 0))
-    (property "Footprint" "hellen-one-common:SOD-323" (id 2) (at 120.65 356.87 0)
-      (effects (font (size 1.27 1.27)) hide)
-    )
-    (property "Datasheet" "" (id 3) (at 123.19 347.98 0)
-      (effects (font (size 1.27 1.27)) hide)
-    )
-    (property "LCSC" "C2128" (id 4) (at 123.19 350.52 0)
+    (property "Value" "1N4148WS" (id 1) (at 116.84 354.33 0))
+    (property "Footprint" "hellen-one-common:SOD-323" (id 2) (at 123.19 344.17 0)
+      (effects (font (size 1.27 1.27)) hide)
+    )
+    (property "Datasheet" "" (id 3) (at 120.65 353.06 0)
+      (effects (font (size 1.27 1.27)) hide)
+    )
+    (property "LCSC" "C2128" (id 4) (at 120.65 350.52 0)
       (effects (font (size 1.27 1.27)) hide)
     )
@@
     (pin "1")
   )
-  (symbol (lib_id "hellen-one-common:1N4148WS") (at 123.19 328.93 0) (mirror y) (unit 1)
-    (in_bom yes) (on_board yes)
-    (property "Reference" "D1" (id 0) (at 125.73 331.47 0))
-    (property "Value" "1N4148WS" (id 1) (at 127 334.01 0))
-    (property "Footprint" "hellen-one-common:SOD-323" (id 2) (at 120.65 335.28 0)
-      (effects (font (size 1.27 1.27)) hide)
-    )
-    (property "Datasheet" "" (id 3) (at 123.19 326.39 0)
-      (effects (font (size 1.27 1.27)) hide)
-    )
-    (property "LCSC" "C2128" (id 4) (at 123.19 328.93 0)
-      (effects (font (size 1.27 1.27)) hide)
-    )
+  (symbol (lib_id "hellen-one-common:1N4148WS") (at 120.65 328.93 0) (mirror x) (unit 1)
+    (in_bom yes) (on_board yes)
+    (property "Reference" "D1" (id 0) (at 118.11 326.39 0))
+    (property "Value" "1N4148WS" (id 1) (at 121.92 332.74 0))
+    (property "Footprint" "hellen-one-common:SOD-323" (id 2) (at 123.19 322.58 0)
+      (effects (font (size 1.27 1.27)) hide)
+    )
+    (property "Datasheet" "" (id 3) (at 120.65 331.47 0)
+      (effects (font (size 1.27 1.27)) hide)
+    )
+    (property "LCSC" "C2128" (id 4) (at 120.65 328.93 0)
+      (effects (font (size 1.27 1.27)) hide)
+    )

Commit message: Upd SCH
Parts:
- removed C18: 22u, hellen-one-common:C0603, symbol hellen-one-common:Cap
- removed C3, C4: 100n, hellen-one-common:C0603, symbol hellen-one-common:Cap
- removed J2: Cortex_Debug, hellen-one-common:PinHeader_2x05_P1.27mm_Vertical_SMD, symbol Connector_Generic:Conn_02x05_Odd_Even
- removed J5, J6: Conn_01x01, TestPoint:TestPoint_Pad_D2.0mm, symbol Connector_Generic:Conn_01x01
- removed J9: Micro_SD_Card, Connector_Card:microSD_HC_Wuerth_693072010801, symbol Connector:Micro_SD_Card
- removed M4: Module-ign8-0.2, hellen-one-ign8-0.2:ign8, symbol hellen-one-ign8-0.1:Module-ign8-0.1
- removed unit 1 of M5
- removed unit 3 of M5
- removed unit 2 of M5
- removed M6: Module-mcu144-0.6, hellen-one-mcu-0.6:mcu, symbol hellen-one-mcu-0.5:Module-mcu-0.5
- removed M7: Module-can-0.1, hellen-one-can-0.1:can, symbol hellen-one-can-0.1:Module-can-0.1
- removed Q18: AO3401A, hellen-one-common:SOT-23, symbol hellen-one-common:MOSFET-P
- removed Q19: AO3400A, hellen-one-common:SOT-23, symbol hellen-one-common:MOSFET-N
- removed R38, R39, R46: 4.7k, hellen-one-common:R0603, symbol hellen-one-common:Res
- removed R96: 33k, hellen-one-common:R0603, symbol hellen-one-common:Res
- removed S1, S2: Button_SPST, hellen-one-common:SMD-2_2.9x3.9x1.7, symbol hellen-one-common:Button_SPST
- removed U4: JDY-33, alphax-2ch:JDY-33, symbol JDY-33:JDY-33
- removed U7: SN74LVC1G06DBVR, Package_TO_SOT_SMD:SOT-23-5, symbol 74xGxx:74LVC1G06
- added C?: 100n, hellen-one-common:C0603, symbol hellen-one-common:Cap
- added J?: Cortex_Debug, hellen-one-common:PinHeader_2x05_P1.27mm_Vertical_SMD, symbol Connector_Generic:Conn_02x05_Odd_Even
- added M10: Module-mega-mcu144-0.2, hellen-one-mega-mcu144-0.2:mega-mcu144, symbol mega-mcu144:Module-mega-mcu144-0.2
- added U?: JDY-33, alphax-2ch:JDY-33, symbol JDY-33:JDY-33
Connections:
- net +3V3: now also J?.1 (Pin_1)
- net +5V: now also M10.N31 (VCC)
- net +5VA: now also M10.E38 (V5A_SWITCHABLE), M10.N30 (V5A_SWITCHABLE), M10.W2 (V5A_SWITCHABLE)
- net 2STEP_PULLDOWN: now also M10.E23 (OUT_IO7)
- net BOOST: now also M10.E16 (OUT_PWM3)
- net BT_3V3: now also C?.2, M10.N28 (V33_SWITCHABLE), U?.12 (3V3)
- net CAM_PULLDOWN: now also M10.E22 (OUT_IO8)
- net CAM_VR_PULLUP: now also M10.E11 (OUT_IO9)
- net CAN+: now also M10.W12 (CANH)
- net CAN-: now also M10.W13 (CANL)
- net CRANK_N_PULLUP: now also M10.E7 (OUT_IO5)
- net CRANK_P_PULLUP: now also M10.E12 (OUT_IO2)
- net D2_PULLDOWN: now also M10.E31 (OUT_INJ5)
- net D3_PULLDOWN: now also M10.E32 (OUT_INJ6)
- net D4_PULLDOWN: now also M10.E33 (OUT_INJ7)
- net D5_PULLDOWN: now also M10.E34 (OUT_INJ8)
- net ETB_DIR: now also M10.N16 (IO1)
- net ETB_DIS: now also M10.N19 (IO2)
- net ETB_PWM: now also M10.E17 (OUT_PWM2)
- net FAN_RELAY: now also M10.E24 (OUT_IO11)
- net GND: now also C?.1, J?.3 (Pin_3), J?.5 (Pin_5), J?.9 (Pin_9), M10.G (GND), U?.13 (GND)
- net GNDA: now also M10.E39 (GNDA), M10.W1 (GNDA)
- net HALL1: now also M10.S4 (IN_D1)
- net HALL2: now also M10.S2 (IN_D3)
- net HALL3: now also M10.S1 (IN_D4)
- net IDLE1: now also M10.E27 (OUT_PWM1)
- net IDLE2: now also M10.E14 (OUT_PWM5)
- net INJ1: now also M10.E19 (OUT_INJ1)
- net INJ2: now also M10.E18 (OUT_INJ2)
- net INJ3: now also M10.E29 (OUT_INJ3)
- net INJ4: now also M10.E30 (OUT_INJ4)
- net IN_2STEP: now also M10.S25 (IN_VSS)
- net IN_AFR: now also M10.S15 (IN_O2S2)
- net IN_CAM_HALL: now also M10.S24 (IN_CAM)
- net IN_CAM_VR: now also M10.S17 (IN_RES1)
- net IN_CLT: now also M10.S28 (IN_CLT)
- net IN_CRANK: now also M10.S22 (IN_CRANK)
- net IN_D2: now also M10.S9 (IN_SENS1)
- net IN_D3: now also M10.S8 (IN_SENS2)
- net IN_D4: now also M10.S7 (IN_SENS3)
- net IN_D5: now also M10.S6 (IN_SENS4)
- net IN_FLEX: now also M10.S10 (IN_AUX4)
- net IN_IAT: now also M10.S26 (IN_IAT)
- net IN_KNOCK: now also M10.S23 (IN_KNOCK)
- net IN_MAP2: now also M10.S20 (IN_MAP2)
- net IN_MAP3: now also M10.S19 (IN_MAP3)
- net IN_PPS1: now also M10.S31 (IN_PPS)
- net IN_PPS2: now also M10.S12 (IN_AUX2)
- net IN_TPS1: now also M10.S30 (IN_TPS)
- net IN_TPS2: now also M10.S13 (IN_AUX1)
- net MAIN: now also M10.E10 (OUT_IO10)
- net NOS: now also M10.E9 (OUT_IO6)
- net NRESET: now also J?.10 (Pin_10), M10.N9 (nReset)
- net OUT_IGN1: now also M10.W11 (IGN1)
- net OUT_IGN2: now also M10.W10 (IGN2)
- net OUT_IGN3: now also M10.W9 (IGN3)
- net OUT_IGN4: now also M10.W8 (IGN4)
- net PUMP_RELAY: now also M10.E13 (OUT_IO12)
- net PWR_EN: now also M10.N29 (OUT_PWR_EN)
- net SWCLK: now also J?.4 (Pin_4), M10.N8 (SWCLK)
- net SWDIO: now also J?.2 (Pin_2), M10.N7 (SWDIO)
- net SWO: now also J?.6 (Pin_6), M10.N6 (SWO)
- net TACH: now also M10.E20 (OUT_IO13)
- net TACH_PULLUP: now also M10.E8 (OUT_IO1)
- net TEMP_PULLUP: now also M10.E21 (OUT_IO4)
- net THRESHOLD_VR_CM: now also M10.E15 (OUT_PWM4)
- net THRESHOLD_VR_CR: now also M10.E26 (OUT_PWM6)
- net TLS115_PG: now also M10.S3 (IN_D2)
- net UART_RX: now also M10.N18 (UART2_RX), U?.1 (TXD)
- net UART_TX: now also M10.N17 (UART2_TX), U?.2 (RXD)
- net USB+: now also M10.N3 (USBP)
- net USB-: now also M10.N2 (USBM)
- net VBUS: now also M10.N4 (VBUS)
- net VIGN: now also M10.N26 (IN_VIGN)
- net VREF2: now also M10.S5 (VREF2)
- net VR_ANALOG_CM: now also M10.S14 (IN_RES2)
- net VR_ANALOG_CR: now also M10.S18 (IN_RES3)
- net VVT1: now also M10.E25 (OUT_PWM7)
- net VVT2: now also M10.E28 (OUT_PWM8)
- no-connect marks 74 -> 62
Other:
- note added: "Сделать без input"
- note removed: "EINT1"
- note removed: "EINT11"
- note removed: "EINT12"
- note removed: "EINT13"
- note removed: "EINT14"
- note removed: "EINT15"
- note removed: "EINT2"
- note removed: "EINT9"
- moved on the sheet: C2, M5D, U3
