File: alphax_4ch.kicad_sch (KiCad schematic)
At the start: 229 parts, among them J1 USB_B_Mini, J10 Conn_01x01, J11 Conn_01x01, J3 Conn_01x01, J4 Conn_01x01, J7 Conn_01x01, J8 Conn_01x01, M1 Module-power12-0.2, M10 Module-mega-mcu144-0.2, M2 Module-power5-0.2, M3 Module-vr-discrete-0.4, M5 Module-input-0.1, M8 Module-vr-discrete-0.4, M9 Module-knock-0.2, P1 33311-24AW-2, P2 33311-24AW-2, Q1 AO3400A, Q10 AO3400A, Q11 AO3400A, Q12 AO3400A, Q13 AO3401A, Q14 AO3401A, Q15 AO3400A, Q16 AO3401A, Q17 AO3401A, Q2 AO3400A, Q20 AO3400A, Q21 AO3400A, Q22 VND14NV04-E, Q23 VND14NV04-E, Q24 AO3400A, Q25 AO3400A, Q26 VND14NV04-E, Q27 AO3400A, Q28 VND14NV04-E, Q29 VND14NV04-E, Q3 AO3401A, Q30 VND14NV04-E, Q31 AO3401A, Q32 AO3401A, Q33 AO3400A, Q34 AO3400A, Q35 AO3400A, Q36 AO3400A, Q4 AO3401A, Q5 AO3401A, Q6 VND14NV04-E, Q7 VND14NV04-E, Q8 VND14NV04-E, Q9 VND14NV04-E, U1 TLS115, U2 74HC2G17GW, U3 MPXH6400A, U5 74HC2G17GW, U6 TLE9201SG

Commit message: Upd SCH
Parts:
- removed C1: 1u, hellen-one-common:C0603, symbol hellen-one-common:Cap
- removed J1: USB_B_Mini, hellen-one-common:USB-MINI-B-HORIZONTAL, symbol hellen-one-common:USB_B_Mini
- removed M1: Module-power12-0.2, hellen-one-power12-0.2:power12, symbol hellen-one-power12-0.2:Module-power12-0.2
- removed M2: Module-power5-0.2, hellen-one-power5-0.2:power5, symbol hellen-one-power5-0.2:Module-power5-0.2
- removed R3: 4.7k, hellen-one-common:R0603, symbol hellen-one-common:Res
- removed R90: 10k, hellen-one-common:R0603, symbol Device:R
- removed U1: TLS115, hellen-one-common:PG-TSON-10-2, symbol hellen-one-common:TLS115
- added J?: Conn_01x05_Male, Connector_Molex:Molex_SPOX_5267-05A_1x05_P2.50mm_Vertical, symbol Connector:Conn_01x05_Male
- added J?: USB_C_Receptacle_USB2.0, Connector_USB:USB_C_Receptacle_XKB_U262-16XN-4BVC11, symbol Connector:USB_C_Receptacle_USB2.0
- added M?: Module-ign8-0.2, hellen-one-ign8-0.2:ign8, symbol hellen-one-ign8-0.2:Module-ign8-0.2
- added M?: Module-power_12and5V-0.1, hellen-one-power_12and5V-0.1:power_12and5V, symbol power_12and5V-0.1:Module-power_12and5V-0.1
- added R90: 10k, hellen-one-common:R0603, symbol hellen-one-common:Res
- added R? (x2): 5.6k, hellen-one-common:R0603, symbol hellen-one-common:Res
Connections:
- net +12V: now also M?.E2 (V12)
- net +12V_RAW: now also M?.V1 (V12_PERM), M?.V3 (V12_RAW)
- net +3V3: now also M10.N22 (V33), R90.2
- net +5V: now also M?.E4 (V5)
- net +5VA: now also M?.V9 (VCC)
- net +5VAS: now also M?.V4 (5VP)
- net BOOST: now also M?.S1 (OUT_IGN8); no longer M10.E16 (OUT_PWM3)
- net BT_3V3: now also M?.V10 (V33)
- net ETB_DIS: now also R90.1
- net FAN_RELAY: now also M?.S4 (OUT_IGN5); no longer M10.E24 (OUT_IO11)
- net GND: now also J?.4 (Pin_4), J?.5 (Pin_5), J?.A1 (GND), J?.A12 (GND), J?.B1 (GND), J?.B12 (GND), J?.S1 (SHIELD), M?.G (GND), M?.S1 (GND), R?.1, R?.1
- net IDLE1: now also M?.S3 (OUT_IGN6); no longer M10.E27 (OUT_PWM1)
- net IDLE2: now also M?.S2 (OUT_IGN7); no longer M10.E14 (OUT_PWM5)
- net INJ1: now also M?.S8 (OUT_IGN1); no longer M10.E19 (OUT_INJ1)
- net INJ2: now also M?.S7 (OUT_IGN2); no longer M10.E18 (OUT_INJ2)
- net INJ3: now also M?.S6 (OUT_IGN3); no longer M10.E29 (OUT_INJ3)
- net INJ4: now also M?.S5 (OUT_IGN4); no longer M10.E30 (OUT_INJ4)
- net IN_VIGN: now also M?.V2 (IN_VIGN)
- net PWR_EN: now also M?.E5 (EN_5VP)
- net TLS115_PG: now also M?.E6 (PG_5VP)
- net USB+: now also J?.3 (Pin_3), J?.A6 (D+), J?.B6 (D+)
- net USB-: now also J?.2 (Pin_2), J?.A7 (D-), J?.B7 (D-)
- net VBUS: now also J?.1 (Pin_1), J?.A4 (VBUS), J?.A9 (VBUS), J?.B4 (VBUS), J?.B9 (VBUS)
- net VIGN: now also M?.E3 (VIGN)
- net VVT1: now also M10.W5 (IGN7); no longer M10.E25 (OUT_PWM7)
- net VVT2: now also M10.W4 (IGN8); no longer M10.E28 (OUT_PWM8)
- new net: J?.A5 (CC1), R?.2
- new net: J?.B5 (CC2), R?.2
- new net MCU_BOOST: M10.E16 (OUT_PWM3), M?.V1 (IGN8)
- new net MCU_FAN_RELAY: M10.E24 (OUT_IO11), M?.V4 (IGN5)
- new net MCU_IDLE1: M10.E27 (OUT_PWM1), M?.V3 (IGN6)
- new net MCU_IDLE2: M10.E14 (OUT_PWM5), M?.V2 (IGN7)
- new net MCU_INJ1: M10.E19 (OUT_INJ1), M?.V8 (IGN1)
- new net MCU_INJ2: M10.E18 (OUT_INJ2), M?.V7 (IGN2)
- new net MCU_INJ3: M10.E29 (OUT_INJ3), M?.V6 (IGN3)
- new net MCU_INJ4: M10.E30 (OUT_INJ4), M?.V5 (IGN4)
- no-connect marks 62 -> 64
Other:
- note added: "* Warning! Remove R40 if you use TLS115"
- note removed: "* Warning! Remove R40 is you use TLS115"
- note removed: "Protected 5V analog power supply for Sensors"
- moved on the sheet: M5D, R40

Commit message: Upd SCH
Parts:
- removed J7, J8: Conn_01x01, MountingHole:MountingHole_4.5mm_Pad, symbol Connector_Generic:Conn_01x01
- removed M10: Module-mega-mcu144-0.2, hellen-one-mega-mcu144-0.2:mega-mcu144, symbol mega-mcu144:Module-mega-mcu144-0.2
- added C1: 470uF, Capacitor_SMD:CP_Elec_10x10.5, symbol Device:C_Polarized
- added C18, C4: 10n, hellen-one-common:C0603, symbol hellen-one-common:Cap
- added D60, D61, D62, D63: B5819W, hellen-one-common:SOD-123, symbol hellen-one-common:1N4148WS
- added J6: 430451012, Connector_Molex:Molex_Micro-Fit_3.0_43045-1012_2x05_P3.00mm_Vertical, symbol Connector_Generic:Conn_02x05_Odd_Even
- added M4: Module-mega-mcu144-0.3, hellen-one-mega-mcu144-0.3:mega-mcu144, symbol mega-mcu144:Module-mega-mcu144-0.3
- added M6: Module-ign8-0.2, hellen-one-ign8-0.2:ign8, symbol hellen-one-ign8-0.2:Module-ign8-0.2
- added P10, P11, P12, P13, P14, P15, P3, P4, P5, P6, P7, P8, P9: Pad, hellen-one-common:PAD-TH, symbol hellen-one-common:Pad
- added Q18, Q39: PJM2319PSA, Package_TO_SOT_SMD:SOT-23, symbol Transistor_FET:IRLML5203
- added Q19, Q40: AO3400A, hellen-one-common:SOT-23, symbol hellen-one-common:MOSFET-N
- added Q37, Q38: VND14NV04-E, hellen-one-common:DPAK, symbol Power_Management:AUIPS2041L
- added R13, R14, R20, R38: DNP, hellen-one-common:R0603, symbol hellen-one-common:Res
- added R39, R66, R7, R71, R96, R97: 4.7k, hellen-one-common:R0603, symbol hellen-one-common:Res
- added R46, R57, R58, R65: 680k, hellen-one-common:R0603, symbol hellen-one-common:Res
- gave numbers to parts that had none: 9
Connections:
- net +12V_ETB: now also C1.1
- net +12V_RAW: now also D62.1 (K), D63.1 (K), Q18.2 (S), Q39.2 (S), R66.2, R7.2
- net +3V3: now also M4.N22 (V33)
- net +5V: now also M4.N31 (VCC)
- net +5VA: now also M4.E38 (V5A_SWITCHABLE), M4.N30 (V5A_SWITCHABLE), M4.W2 (V5A_SWITCHABLE), M6.V9 (VCC), R13.2, R14.2, R20.2, R38.2
- net 2STEP_PULLDOWN: now also M4.E23 (OUT_IO7)
- net BT_3V3: now also M4.N28 (V33_SWITCHABLE), M6.V10 (V33)
- net CAM_PULLDOWN: now also M4.E22 (OUT_IO8)
- net CAM_VR_PULLUP: now also M4.E11 (OUT_IO9)
- net CAN+: now also M4.W12 (CANH)
- net CAN-: now also M4.W13 (CANL)
- net CRANK_N_PULLUP: now also M4.E7 (OUT_IO5)
- net CRANK_P_PULLUP: now also M4.E12 (OUT_IO2)
- net D2_PULLDOWN: now also M4.E31 (OUT_INJ5)
- net D3_PULLDOWN: now also M4.E32 (OUT_INJ6)
- net D4_PULLDOWN: now also M4.E33 (OUT_INJ7)
- net D5_PULLDOWN: now also M4.E34 (OUT_INJ8)
- net ETB_DIR: now also M4.N16 (IO1)
- net ETB_DIS: now also M4.N19 (IO2)
- net ETB_PWM: now also M4.E17 (OUT_PWM2)
- net GND: now also C1.2, C18.1, C4.1, D60.2 (A), D61.2 (A), M4.G (GND), M6.G (GND), M6.V1 (IGN8), M6.V2 (IGN7), M6.V3 (IGN6), M6.V4 (IGN5), M6.V5 (IGN4), M6.V6 (IGN3), Q19.3 (S), Q37.3 (S), Q38.3 (S), Q40.3 (S), R39.2, R71.2, R96.2, R97.2
- net GNDA: now also M4.E39 (GNDA), M4.W1 (GNDA), R46.1, R57.1, R58.1, R65.1
- net HALL1: now also M4.S4 (IN_D1)
- net HALL2: now also M4.S2 (IN_D3)
- net HALL3: now also M4.S1 (IN_D4)
- net IN_2STEP: now also M4.S25 (IN_VSS)
- net IN_AFR: now also M4.S15 (IN_O2S2)
- net IN_CAM_HALL: now also M4.S24 (IN_CAM)
- net IN_CAM_VR: now also M4.S17 (IN_RES1)
- net IN_CLT: now also M4.S28 (IN_CLT)
- net IN_CRANK: now also M4.S22 (IN_CRANK)
- net IN_D2: now also M4.S9 (IN_SENS1)
- net IN_D3: now also M4.S8 (IN_SENS2)
- net IN_D4: now also M4.S7 (IN_SENS3)
- net IN_D5: now also M4.S6 (IN_SENS4)
- net IN_FLEX: now also M4.S10 (IN_AUX4)
- net IN_IAT: now also M4.S26 (IN_IAT)
- net IN_KNOCK: now also M4.S23 (IN_KNOCK)
- net IN_MAP2: now also M4.S20 (IN_MAP2)
- net IN_MAP3: now also M4.S19 (IN_MAP3)
- net IN_PPS1: now also M4.S31 (IN_PPS)
- net IN_PPS2: now also M4.S12 (IN_AUX2)
- net IN_TPS1: now also M4.S30 (IN_TPS)
- net IN_TPS2: now also M4.S13 (IN_AUX1)
- net MAIN: now also M4.E10 (OUT_IO10)
- net MCU_BOOST: now also M4.E16 (OUT_PWM3)
- net MCU_FAN_RELAY: now also M4.E24 (OUT_IO11)
- net MCU_IDLE1: now also M4.E27 (OUT_PWM1)
- net MCU_IDLE2: now also M4.E14 (OUT_PWM5)
- net MCU_INJ1: now also M4.E19 (OUT_INJ1)
- net MCU_INJ2: now also M4.E18 (OUT_INJ2)
- net MCU_INJ3: now also M4.E29 (OUT_INJ3)
- net MCU_INJ4: now also M4.E30 (OUT_INJ4)
- net NOS: now also M4.E9 (OUT_IO6)
- net NRESET: now also M4.N9 (nReset)
- net OUT_ETB+: now also C18.2
- net OUT_ETB-: now also C4.2
- net OUT_IGN1: now also M4.W11 (IGN1)
- net OUT_IGN2: now also M4.W10 (IGN2)
- net OUT_IGN3: now also M4.W9 (IGN3)
- net OUT_IGN4: now also M4.W8 (IGN4)
- net PUMP_RELAY: now also M4.E13 (OUT_IO12)
- net PWR_EN: now also M4.N29 (OUT_PWR_EN)
- net SWCLK: now also M4.N8 (SWCLK)
- net SWDIO: now also M4.N7 (SWDIO)
- net SWO: now also M4.N6 (SWO)
- net TACH: now also M4.E20 (OUT_IO13)
- net TACH_PULLUP: now also M4.E8 (OUT_IO1)
- net TEMP_PULLUP: now also M4.E21 (OUT_IO4)
- net THRESHOLD_VR_CM: now also M4.E15 (OUT_PWM4)
- net THRESHOLD_VR_CR: now also M4.E26 (OUT_PWM6)
- net TLS115_PG: now also M4.S3 (IN_D2)
- net UART_RX: now also M4.N18 (UART2_RX)
- net UART_TX: now also M4.N17 (UART2_TX)
- net USB+: now also M4.N3 (USBP)
- net USB-: now also M4.N2 (USBM)
- net VBUS: now also M4.N4 (VBUS)
- net VIGN: now also M4.N26 (IN_VIGN)
- net VREF2: now also M4.S5 (VREF2)
- net VR_ANALOG_CM: now also M4.S14 (IN_RES2)
- net VR_ANALOG_CR: now also M4.S18 (IN_RES3)
- net VVT1: now also M4.W5 (IGN7)
- net VVT2: now also M4.W4 (IGN8)
- new net: M4.E1 (SPI2_SCK), P5.1 (Pin_1)
- new net: M4.E2 (SPI2_MISO), P6.1 (Pin_1)
- new net: M4.E3 (SPI2_MOSI), P7.1 (Pin_1)
- new net: M4.E35 (IO6), P14.1 (Pin_1)
- new net: M4.E36 (IO7), P15.1 (Pin_1)
- new net: M4.E4 (SPI2_CS), P8.1 (Pin_1)
- new net: M4.E6 (OUT_IO3), P10.1 (Pin_1)
- new net: M4.N14 (I2C_SCL), P13.1 (Pin_1)
- new net: M4.N15 (I2C_SDA), P12.1 (Pin_1)
- new net: M4.S27 (IN_AT1), P11.1 (Pin_1)
- new net: Q39.1 (G), Q40.2 (D), R66.1
- new net: Q18.1 (G), Q19.2 (D), R7.1
- new net AIN1: J6.1 (Pin_1), M4.S32 (IN_TPS2), R13.1, R46.2
- new net AIN2: J6.3 (Pin_3), M4.S33 (IN_PPS2), R14.1, R57.2
- new net AIN3: J6.5 (Pin_5), M4.S21 (IN_MAP1), R20.1, R58.2
- new net AIN4: J6.7 (Pin_7), M4.S11 (IN_AUX3), R38.1, R65.2
- new net HS1: M4.E25 (OUT_PWM7), Q19.1 (G), R39.1
- new net HS2: M4.E28 (OUT_PWM8), Q40.1 (G), R97.1
- new net INJ5: M6.S8 (OUT_IGN1), Q37.1 (IN), R71.1
- new net INJ6: M6.S7 (OUT_IGN2), Q38.1 (IN), R96.1
- new net MCU_INJ5: M6.V8 (IGN1)
- new net MCU_INJ6: M6.V7 (IGN2)
- new net OUT_HS1: D60.1 (K), J6.9 (Pin_9), Q18.3 (D)
- new net OUT_HS2: D61.1 (K), J6.10 (Pin_10), Q39.3 (D)
- new net OUT_IGN5: J6.6 (Pin_6), M4.W7 (IGN5), P3.1 (Pin_1)
- new net OUT_IGN6: J6.8 (Pin_8), M4.W6 (IGN6), P4.1 (Pin_1)
- new net OUT_INJ5: D62.2 (A), J6.2 (Pin_2), Q37.2 (D)
- new net OUT_INJ6: D63.2 (A), J6.4 (Pin_4), Q38.2 (D)
- no-connect marks 64 -> 57
Other:
- note added: "AUX"
- moved on the sheet: C10, C11, C12, C13, C14, C15, C16, C2, C6, C7, C8, C9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

Commit message: Upd SCH
Parts:
- removed C1: 470uF, Capacitor_SMD:CP_Elec_10x10.5, symbol Device:C_Polarized
- removed C10, C11, C12, C13, C14, C15, C16, C7, C8, C9: 10u, hellen-one-common:C0805, symbol Device:C
- removed C17, C2, C3, C5: 100n, hellen-one-common:C0603, symbol hellen-one-common:Cap
- removed C18, C4: 10n, hellen-one-common:C0603, symbol hellen-one-common:Cap
- removed C6: 100n, hellen-one-common:C0603, symbol Device:C
- removed D25, D26, D27, D28, D29, D50, D51, D52, D53, D54, D56, D60, D61, D62, D63: B5819W, hellen-one-common:SOD-123, symbol hellen-one-common:1N4148WS
- removed D49: PSM712-LF, hellen-one-common:SOT-23, symbol Power_Management:PSM712
- removed D55: PSM712-LF, hellen-one-common:SOT-23, symbol hellen-one-common:PSM712
- removed D57, D58, D59: BAT54S, Package_TO_SOT_SMD:SOT-23, symbol Diode:BAT54S
- removed J1: USB_C_Receptacle_USB2.0, Connector_USB:USB_C_Receptacle_XKB_U262-16XN-4BVC11, symbol Connector:USB_C_Receptacle_USB2.0
- removed J2: Conn_01x05_Male, Connector_Molex:Molex_SPOX_5267-05A_1x05_P2.50mm_Vertical, symbol Connector:Conn_01x05_Male
- removed J5: Cortex_Debug, hellen-one-common:PinHeader_2x05_P1.27mm_Vertical_SMD, symbol Connector_Generic:Conn_02x05_Odd_Even
- removed M4: Module-mega-mcu144-0.3, hellen-one-mega-mcu144-0.3:mega-mcu144, symbol mega-mcu144:Module-mega-mcu144-0.3
- removed M5: Module-input-0.1, hellen-one-input-0.1:input, symbol hellen-one-input-0.1:Module-input-0.1
- removed P10, P11, P12, P13, P14, P15, P3, P4, P5, P6, P7, P8, P9: Pad, hellen-one-common:PAD-TH, symbol hellen-one-common:Pad
- removed Q1, Q10, Q11, Q12, Q15, Q19, Q2, Q20, Q21, Q24, Q25, Q27, Q33, Q34, Q35, Q36, Q40: AO3400A, hellen-one-common:SOT-23, symbol hellen-one-common:MOSFET-N
- removed Q13, Q14, Q16, Q17, Q3, Q31, Q32, Q4, Q5: AO3401A, hellen-one-common:SOT-23, symbol hellen-one-common:MOSFET-P
- removed Q18, Q39: PJM2319PSA, Package_TO_SOT_SMD:SOT-23, symbol Transistor_FET:IRLML5203
- removed Q22, Q23, Q26, Q28, Q29, Q30, Q37, Q38, Q6, Q7, Q8, Q9: VND14NV04-E, hellen-one-common:DPAK, symbol Power_Management:AUIPS2041L
- removed R14, R20, R38: DNP, hellen-one-common:R0603, symbol hellen-one-common:Res
- removed R21, R23, R34, R36, R77: 2k, hellen-one-common:R1206, symbol hellen-one-common:Res
- removed R25, R26, R27, R28, R78, R83, R84: 4.7k, hellen-one-common:R0603-4, symbol hellen-one-common:Res_Array_4
- removed R29, R42, R79, R80, R81, R82: 1.2k, hellen-one-common:R0603, symbol hellen-one-common:Res
- removed R3, R6: 5.6k, hellen-one-common:R0603, symbol hellen-one-common:Res
- removed R30, R31, R39, R41, R43, R66, R7, R71, R92, R96, R97: 4.7k, hellen-one-common:R0603, symbol hellen-one-common:Res
- removed R32, R33: 2.7k, hellen-one-common:R0603, symbol hellen-one-common:Res
- removed R44, R45, R86, R87, R88: 3.3k, hellen-one-common:R0603, symbol hellen-one-common:Res
- removed R47: 470, hellen-one-common:R0805, symbol hellen-one-common:Res
- removed R57, R58, R65: 680k, hellen-one-common:R0603, symbol hellen-one-common:Res
- removed R90: 10k, hellen-one-common:R0603, symbol hellen-one-common:Res
- removed R94, R95: 510k, hellen-one-common:R0603, symbol hellen-one-common:Res
- removed U1: JDY-33, alphax-2ch:JDY-33, symbol JDY-33:JDY-33
- removed U2, U5: 74HC2G17GW, hellen-one-common:SOT-363, symbol 74xGxx:74LVC2G17
- removed U3: MPXH6400A, hellen-one-common:MPXH6400A-SSOP8, symbol MPX-4_MAP:MPX4_MAP
- removed U6: TLE9201SG, Package_SO:Infineon_PG-DSO-12-11, symbol rusefi_tle9201:TLE9201SG
- R48: value 4.7k -> DNP; LCSC C23162 -> (none)
- R74, R76, R93: value 4.7k -> 680k; LCSC C23162 -> C25822
- R75: value 2k -> DNP; footprint hellen-one-common:R1206 -> hellen-one-common:R0603; LCSC C17944 -> (none)
- R89: value 3.3k -> DNP; LCSC C22978 -> (none)
Connections:
- net +5VA: now also R48.2, R75.2, R89.2
- net AIN2: now also R48.1, R74.2
- net AIN3: now also R75.1, R76.2
- net AIN4: now also R89.1, R93.2
- net CAM_VR_PULLUP: no longer R74.1
- net GND: no longer R74.2
- net GNDA: now also R74.1, R76.1, R93.1
- net HALL1: now also R24.1
- net HALL2: now also R37.1
- net HALL3: now also R73.1
- net IN_CAM_VR+: no longer R75.2
- net IN_D5: no longer R89.1
- net IN_MAP2: no longer R19.1
- net BT_3V3 renamed +3.3VA
- new net IN_MAP: R19.1
- no-connect marks 57 -> 9
Other:
- added sheet ETB (ETB.kicad_sch)
- added sheet HALL_OPT_PU (HALL_PU3.kicad_sch)
- added sheet HS (HS2.kicad_sch)
- added sheet INJ (INJ4.kicad_sch)
- added sheet LS1 (LS4.kicad_sch)
- added sheet LS2 (LS4.kicad_sch)
- added sheet LS_weak (LS_weak.kicad_sch)
- added sheet MAP (MAP.kicad_sch)
- added sheet MCU (MCU.kicad_sch)
- added sheet OPT_PULLDOWNS1 (PD4.kicad_sch)
- added sheet OPT_PULLDOWNS2 (PD2.kicad_sch)
- added sheet OPT_PULLUPS (DOUBLE_PU.kicad_sch)
- added sheet TACH_PULLUP (TACH_PU.kicad_sch)
- note removed: "4k pullups"
- note removed: "Bluetooth Module"
- note removed: "CRANK/CAM test pads"
- note removed: "EINT3"
- note removed: "EINT4"
- note removed: "EINT5"
- note removed: "EINT6"
- note removed: "EINT7"
- note removed: "ETB driver"
- note removed: "HALL sensor inputs"
- note removed: "Internal MAP"
- note removed: "MCU Debug Port"
- note removed: "Outputs"
- note removed: "Pullups / Pulldowns"
- note removed: "Wake-up pin:"
- note removed: "Сделать без input"
- moved on the sheet: D1, D10, D11, D12, D13, D14, D15, D16, D17, D18, D19, D2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

Commit message: Upd PCB
Parts:
- removed D18, D19, D23, D24: LED-BLUE-0603, hellen-one-common:LED-0603, symbol hellen-one-common:LED_0603
- removed M3, M8: Module-vr-discrete-0.4, hellen-one-vr-discrete-0.4:vr-discrete, symbol vr-discrete-0.4:Module-vr-discrete-0.4
- removed R4: 1k, hellen-one-common:R0603-4, symbol hellen-one-common:Res_Array_4
- added F10, F11: nSMD005, hellen-one-common:PAD-1206-PAD, symbol hellen-one-common:Fuse-Pad-Pad
- added J7, J8: Conn_01x01, MountingHole:MountingHole_4.5mm_Pad, symbol Connector_Generic:Conn_01x01
- added M3, M8: Module-vr-discrete-0.4, hellen-one-vr-discrete-0.4:vr-discrete, symbol hellen-one-vr-discrete-0.4:Module-vr-discrete-0.4
Connections:
- net +5V: now also M3.E4 (V5_IN), M8.E4 (V5_IN)
- net GND: now also M3.G (GND), M8.G (GND)
- net IN_CAM_VR: now also M3.E3 (OUT)
- net IN_CAM_VR+: now also M3.W2 (VR+)
- net IN_CAM_VR-: now also M3.W1 (VR-)
- net IN_CRANK: now also M8.E3 (OUT)
- net IN_CRANK+: now also M8.W2 (VR+)
- net IN_CRANK-: now also M8.W1 (VR-)
- net OUT_IGN5: now also F10.2; no longer J6.6 (Pin_6)
- net OUT_IGN6: now also F11.2; no longer J6.8 (Pin_8)
- net THRESHOLD_VR_CM: now also M3.E1 (Thresh_IN)
- net THRESHOLD_VR_CR: now also M8.E1 (Thresh_IN)
- net VR_ANALOG_CM: now also M3.E2 (OUT_A)
- net VR_ANALOG_CR: now also M8.E2 (OUT_A)
- new net: F11.1, J6.8 (Pin_8)
- new net: F10.1, J6.6 (Pin_6)
- no-connect marks 9 -> 11
Other:
- sheet MCU ports: added IN_MAP; removed IN_MAP1
- note added: "1.2k UP (default)/4.5k DOWN"
- note added: "12A Low-side (VND14)"
- note added: "3A High-side"
- note added: "5A Low-side"
- note added: "5V 750 Ohm (default)/12V 970 Ohm"
- note added: "Configurable AUX pulls"
- note added: "Float (default)/2.7k UP"
- note added: "Float (default)/4.47k UP"
- note added: "Internal MAP sensor"
- note added: "TLE9201 motor driver"
- note removed: "Auxiliary bus"

Commit message: Fab preview
Parts:
- removed J10, J11: Conn_01x01, TestPoint:TestPoint_Pad_D2.0mm, symbol Connector_Generic:Conn_01x01
- added C17, C20, C21: 1n 250V, hellen-one-common:C0603, symbol hellen-one-common:Cap
- added P3, P4: Pad, hellen-one-common:PAD-TH, symbol hellen-one-common:Pad
- added R39, R4: 4.7k, hellen-one-common:R0603, symbol hellen-one-common:Res
Connections:
- net +12V: now also D20.1 (A), D22.1 (K)
- net +12V_RAW: no longer D20.1 (A), D22.1 (K)
- net +5V: no longer M3.E4 (V5_IN), M8.E4 (V5_IN), R1.1, R1.2, R1.3, R1.4, R50.1, R50.2
- net +5VA: now also M3.E4 (V5_IN), M8.E4 (V5_IN), R1.1, R1.2, R1.3, R1.4, R50.1, R50.2, R39.1, R4.1
- net GND: now also C17.1, C20.1, C21.1
- net IN_2STEP: now also R39.2
- net IN_CAM_HALL: now also P3.1 (Pin_1), R4.2
- net IN_CAM_VR+: now also C21.2
- net IN_CRANK: now also P4.1 (Pin_1)
- net IN_CRANK+: now also C17.2
- net IN_CRANK-: now also C20.2
- net VREF2 renamed VREF
Other:
- sheet MCU ports: added VREF; removed VREF2
- note added: "CAM HALL PU 5VA: remove R21 5VAS configurable: - remove R4"
- note added: "IN_CRANK+ line HALL: remove R753_2"

Commit message: Upd PCB
Parts:
- C20, C21: value 1n 250V -> ~; LCSC C277510 -> (none); MyComment (none) -> DNP
Other:
- note added: "remove 1nf for VR"
Changed lines of the file:
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@@
     (effects (font (size 1.27 1.27)) (justify left bottom))
   )
+  (text "remove 1nf for VR" (at 241.3 179.705 0)
+    (effects (font (size 1.27 1.27)) (justify left bottom))
+  )
   (text "1.2k UP (default)/4.5k DOWN" (at 299.72 280.67 0)
     (effects (font (size 1.27 1.27)) (justify left bottom))
@@
     )
   )
-  (symbol (lib_id "hellen-one-common:Cap") (at 248.92 193.04 0) (mirror x) (unit 1)
-    (in_bom yes) (on_board yes) (dnp no)
-    (property "Reference" "C21" (at 253.365 191.77 0)
-      (effects (font (size 1.27 1.27)) (justify right))
-    )
-    (property "Value" "1n 250V" (at 257.81 194.31 0)
-      (effects (font (size 1.27 1.27)) (justify right))
-    )
-    (property "Footprint" "hellen-one-common:C0603" (at 246.38 189.23 0)
-      (effects (font (size 1.27 1.27)) hide)
-    )
-    (property "Datasheet" "" (at 245.11 193.04 90)
-      (effects (font (size 1.27 1.27)) hide)
-    )
-    (property "LCSC" "C277510" (at 248.92 193.04 0)
-      (effects (font (size 1.27 1.27)) hide)
-    )
-    (pin "1")
-    (pin "2")
-    (instances
-      (project "alphax_4ch"
-        (path "/63d2dd9f-d5ff-4811-a88d-0ba932475460"
-          (reference "C21") (unit 1)
-        )
-        (path "/63d2dd9f-d5ff-4811-a88d-0ba932475460/aafb5e2e-7f5c-429b-85e5-76b90069790c"
-          (reference "C2") (unit 1)
-        )
-      )
-    )
-  )
   (symbol (lib_id "hellen-one-common:Res") (at 250.19 288.29 0) (unit 1)
     (in_bom yes) (on_board yes) (dnp no)
@@
     )
   )
+  (symbol (lib_id "hellen-one-common:Cap") (at 248.92 193.04 0) (mirror x) (unit 1)
+    (in_bom yes) (on_board yes) (dnp no)
+    (property "Reference" "C21" (at 253.365 191.77 0)
+      (effects (font (size 1.27 1.27)) (justify right))
+    )
+    (property "Value" "~" (at 257.81 194.31 0)
+      (effects (font (size 1.27 1.27)) (justify right))
+    )
+    (property "Footprint" "hellen-one-common:C0603" (at 246.38 189.23 0)
+      (effects (font (size 1.27 1.27)) hide)
+    )
+    (property "Datasheet" "" (at 245.11 193.04 90)
+      (effects (font (size 1.27 1.27)) hide)
+    )
+    (property "LCSC" "" (at 248.92 193.04 0)
+      (effects (font (size 1.27 1.27)) hide)
+    )
+    (property "MyComment" "DNP" (at 251.46 194.31 0)
+      (effects (font (size 1.27 1.27)))
+    )
+    (pin "1")
+    (pin "2")
+    (instances
+      (project "alphax_4ch"
+        (path "/63d2dd9f-d5ff-4811-a88d-0ba932475460"
+          (reference "C21") (unit 1)
+        )
+        (path "/63d2dd9f-d5ff-4811-a88d-0ba932475460/aafb5e2e-7f5c-429b-85e5-76b90069790c"
+          (reference "C2") (unit 1)
+        )
+      )
+    )
+  )
   (symbol (lib_id "hellen-one-common:+12V_RAW") (at 34.29 368.3 0) (unit 1)
     (in_bom yes) (on_board yes) (dnp no)
@@
       (effects (font (size 1.27 1.27)) (justify right))
     )
-    (property "Value" "1n 250V" (at 257.81 189.23 0)
+    (property "Value" "~" (at 257.81 189.23 0)
       (effects (font (size 1.27 1.27)) (justify right))
     )
@@
       (effects (font (size 1.27 1.27)) hide)
     )
-    (property "LCSC" "C277510" (at 248.92 187.96 0)
+    (property "LCSC" "" (at 248.92 187.96 0)
       (effects (font (size 1.27 1.27)) hide)
     )
+    (property "MyComment" "DNP" (at 251.46 189.23 0)
+      (effects (font (size 1.27 1.27)))
+    )
     (pin "1")
