File: LS_weak.kicad_sch (KiCad schematic)
At the start: 12 parts, among them Q10 AO3400A, Q11 AO3400A, Q24 AO3400A, Q27 AO3400A

Commit message: Fab preview
Changed lines of the file:
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@@
   (symbol (lib_id "hellen-one-common:1N4148WS") (at 154.94 107.95 0) (unit 1)
     (in_bom yes) (on_board yes) (dnp no)
-    (property "Reference" "D27" (at 156.21 100.33 0)
+    (property "Reference" "D27" (at 156.21 102.235 0)
       (effects (font (size 1.27 1.27)))
     )
