File: ETB.kicad_sch (KiCad schematic)
At the start: 16 parts, among them U6 TLE9201SG

Commit message: Upd PCB
Connections:
- net +3V3 renamed +3.3V
Changed lines of the file:
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@@
         )
         (path "/63d2dd9f-d5ff-4811-a88d-0ba932475460/9d5f2373-d6e9-40ca-9362-36e5ef659bc6"
-          (reference "#PWR0155") (unit 1)
+          (reference "#PWR0110") (unit 1)
         )
       )
@@
         )
         (path "/63d2dd9f-d5ff-4811-a88d-0ba932475460/9d5f2373-d6e9-40ca-9362-36e5ef659bc6"
-          (reference "#PWR0158") (unit 1)
+          (reference "#PWR0105") (unit 1)
         )
       )
@@
         )
         (path "/63d2dd9f-d5ff-4811-a88d-0ba932475460/9d5f2373-d6e9-40ca-9362-36e5ef659bc6"
-          (reference "#PWR084") (unit 1)
+          (reference "#PWR0108") (unit 1)
         )
       )
@@
         )
         (path "/63d2dd9f-d5ff-4811-a88d-0ba932475460/9d5f2373-d6e9-40ca-9362-36e5ef659bc6"
-          (reference "#PWR0163") (unit 1)
+          (reference "#PWR0114") (unit 1)
         )
       )
@@
         )
         (path "/63d2dd9f-d5ff-4811-a88d-0ba932475460/9d5f2373-d6e9-40ca-9362-36e5ef659bc6"
-          (reference "#PWR0168") (unit 1)
+          (reference "#PWR0120") (unit 1)
         )
       )
@@
         )
         (path "/63d2dd9f-d5ff-4811-a88d-0ba932475460/9d5f2373-d6e9-40ca-9362-36e5ef659bc6"
-          (reference "#PWR0164") (unit 1)
+          (reference "#PWR0115") (unit 1)
         )
       )
@@
         )
         (path "/63d2dd9f-d5ff-4811-a88d-0ba932475460/9d5f2373-d6e9-40ca-9362-36e5ef659bc6"
-          (reference "#PWR0150") (unit 1)
+          (reference "#PWR0125") (unit 1)
         )
       )
@@
         )
         (path "/63d2dd9f-d5ff-4811-a88d-0ba932475460/9d5f2373-d6e9-40ca-9362-36e5ef659bc6"
-          (reference "#PWR0151") (unit 1)
+          (reference "#PWR0126") (unit 1)
         )
       )
@@
         )
         (path "/63d2dd9f-d5ff-4811-a88d-0ba932475460/9d5f2373-d6e9-40ca-9362-36e5ef659bc6"
-          (reference "#PWR0159") (unit 1)
+          (reference "#PWR0107") (unit 1)
         )
       )
@@
         )
         (path "/63d2dd9f-d5ff-4811-a88d-0ba932475460/9d5f2373-d6e9-40ca-9362-36e5ef659bc6"
-          (reference "#PWR0161") (unit 1)
+          (reference "#PWR0106") (unit 1)
         )
       )
@@
         )
         (path "/63d2dd9f-d5ff-4811-a88d-0ba932475460/9d5f2373-d6e9-40ca-9362-36e5ef659bc6"
-          (reference "#PWR0160") (unit 1)
+          (reference "#PWR0109") (unit 1)
         )
       )
@@
         )
         (path "/63d2dd9f-d5ff-4811-a88d-0ba932475460/9d5f2373-d6e9-40ca-9362-36e5ef659bc6"
-          (reference "#PWR0165") (unit 1)
+          (reference "#PWR0119") (unit 1)
         )
       )
@@
         )
         (path "/63d2dd9f-d5ff-4811-a88d-0ba932475460/9d5f2373-d6e9-40ca-9362-36e5ef659bc6"
-          (reference "#PWR051") (unit 1)
+          (reference "#PWR0121") (unit 1)
         )
       )
@@
         )
         (path "/63d2dd9f-d5ff-4811-a88d-0ba932475460/9d5f2373-d6e9-40ca-9362-36e5ef659bc6"
-          (reference "#PWR0162") (unit 1)
+          (reference "#PWR0113") (unit 1)
         )
       )
@@
         )
         (path "/63d2dd9f-d5ff-4811-a88d-0ba932475460/9d5f2373-d6e9-40ca-9362-36e5ef659bc6"
-          (reference "#PWR082") (unit 1)
+          (reference "#PWR0123") (unit 1)
         )
       )
@@
         )
         (path "/63d2dd9f-d5ff-4811-a88d-0ba932475460/9d5f2373-d6e9-40ca-9362-36e5ef659bc6"
+          (reference "#PWR0127") (unit 1)
+        )
+      )
+    )
+  )
+  (symbol (lib_id "power:+3.3V") (at 146.05 113.03 270) (unit 1)
+    (in_bom yes) (on_board yes) (dnp no)
+    (property "Reference" "#PWR0162" (at 142.24 113.03 0)
+      (effects (font (size 1.27 1.27)) hide)
+    )
+    (property "Value" "+3.3V" (at 152.4 113.03 90)
+      (effects (font (size 1.27 1.27)))
+    )
+    (property "Footprint" "" (at 146.05 113.03 0)
+      (effects (font (size 1.27 1.27)) hide)
+    )
+    (property "Datasheet" "" (at 146.05 113.03 0)
+      (effects (font (size 1.27 1.27)) hide)
+    )
+    (pin "1")
+    (instances
+      (project "alphax_4ch"
+        (path "/63d2dd9f-d5ff-4811-a88d-0ba932475460"
+          (reference "#PWR0162") (unit 1)
+        )
+        (path "/63d2dd9f-d5ff-4811-a88d-0ba932475460/9d5f2373-d6e9-40ca-9362-36e5ef659bc6"
+          (reference "#PWR0129") (unit 1)
+        )
+      )
+    )
+  )
+  (symbol (lib_id "power:GND") (at 92.71 115.57 0) (unit 1)
+    (in_bom yes) (on_board yes) (dnp no)
+    (property "Reference" "#PWR0152" (at 92.71 121.92 0)
+      (effects (font (size 1.27 1.27)) hide)
+    )
+    (property "Value" "GND" (at 92.7608 119.5134 0)
+      (effects (font (size 1.27 1.27)))
+    )
+    (property "Footprint" "" (at 92.71 115.57 0)
+      (effects (font (size 1.27 1.27)) hide)
+    )
+    (property "Datasheet" "" (at 92.71 115.57 0)
+      (effects (font (size 1.27 1.27)) hide)
+    )
+    (pin "1")
+    (instances
+      (project "alphax_4ch"
+        (path "/63d2dd9f-d5ff-4811-a88d-0ba932475460"
           (reference "#PWR0152") (unit 1)
         )
-      )
-    )
-  )
-  (symbol (lib_id "power:+3.3V") (at 146.05 113.03 270) (unit 1)
-    (in_bom yes) (on_board yes) (dnp no)
-    (property "Reference" "#PWR0162" (at 142.24 113.03 0)
-      (effects (font (size 1.27 1.27)) hide)
-    )
-    (property "Value" "+3.3V" (at 152.4 113.03 90)
-      (effects (font (size 1.27 1.27)))
-    )
-    (property "Footprint" "" (at 146.05 113.03 0)
-      (effects (font (size 1.27 1.27)) hide)
-    )
-    (property "Datasheet" "" (at 146.05 113.03 0)
-      (effects (font (size 1.27 1.27)) hide)
-    )
-    (pin "1")
-    (instances
-      (project "alphax_4ch"
-        (path "/63d2dd9f-d5ff-4811-a88d-0ba932475460"
-          (reference "#PWR0162") (unit 1)
-        )
-        (path "/63d2dd9f-d5ff-4811-a88d-0ba932475460/9d5f2373-d6e9-40ca-9362-36e5ef659bc6"
-          (reference "#PWR0156") (unit 1)
-        )
-      )
-    )
-  )
-  (symbol (lib_id "power:GND") (at 92.71 115.57 0) (unit 1)
-    (in_bom yes) (on_board yes) (dnp no)
-    (property "Reference" "#PWR0152" (at 92.71 121.92 0)
-      (effects (font (size 1.27 1.27)) hide)
-    )
-    (property "Value" "GND" (at 92.7608 119.5134 0)
-      (effects (font (size 1.27 1.27)))
-    )
-    (property "Footprint" "" (at 92.71 115.57 0)
-      (effects (font (size 1.27 1.27)) hide)
-    )
-    (property "Datasheet" "" (at 92.71 115.57 0)
-      (effects (font (size 1.27 1.27)) hide)
-    )
-    (pin "1")
-    (instances
-      (project "alphax_4ch"
-        (path "/63d2dd9f-d5ff-4811-a88d-0ba932475460"
-          (reference "#PWR0152") (unit 1)
-        )
-        (path "/63d2dd9f-d5ff-4811-a88d-0ba932475460/9d5f2373-d6e9-40ca-9362-36e5ef659bc6"
-          (reference "#PWR0166") (unit 1)
+        (path "/63d2dd9f-d5ff-4811-a88d-0ba932475460/9d5f2373-d6e9-40ca-9362-36e5ef659bc6"
+          (reference "#PWR0118") (unit 1)
         )
       )
@@
         )
         (path "/63d2dd9f-d5ff-4811-a88d-0ba932475460/9d5f2373-d6e9-40ca-9362-36e5ef659bc6"
-          (reference "#PWR0154") (unit 1)
-        )
-      )
+          (reference "#PWR0128") (unit 1)
+        )
+      )

Commit message: 10k fix
Parts:
- R90: value 10k -> 4.7k; LCSC C22978 -> C23162
Changed lines of the file:
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@@
       (effects (font (size 1.27 1.27)))
     )
-    (property "Value" "10k" (at 146.05 107.95 0)
+    (property "Value" "4.7k" (at 146.05 107.95 0)
       (effects (font (size 1.27 1.27)))
     )
@@
       (effects (font (size 1.27 1.27)) hide)
     )
-    (property "LCSC" "C22978" (at 146.05 102.87 0)
+    (property "LCSC" "C23162" (at 146.05 102.87 0)
       (effects (font (size 1.27 1.27)) hide)
     )
