File: HALL_PU3.kicad_sch (KiCad schematic)
At the start: 27 parts, among them Q15 AO3400A, Q16 AO3401A, Q17 AO3401A, Q2 AO3400A, Q25 AO3400A, Q31 AO3401A, Q32 AO3401A, Q4 AO3401A, Q5 AO3401A

Commit message: Upd PCB
Parts:
- added D78 (x3): BAT54S, Package_TO_SOT_SMD:SOT-23, symbol Diode:BAT54S
Connections:
- net +12V_LIM: now also D78.2, D78.2, D78.2
- net GND: now also D78.1, D78.1, D78.1
- net at Q32.2 (D), R77.1: now also D78.3
- net at Q17.2 (D), R36.1: now also D78.3
- net at Q5.2 (D), R23.1: now also D78.3
Changed lines of the file:
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@@
   (junction (at 179.07 39.37) (diameter 0) (color 0 0 0 0)
   )
+  (junction (at 125.73 59.69) (diameter 0) (color 0 0 0 0)
+  )
   (junction (at 125.73 99.06) (diameter 0) (color 0 0 0 0)
   )
@@
   (junction (at 160.02 167.64) (diameter 0) (color 0 0 0 0)
   )
+  (junction (at 125.73 109.22) (diameter 0) (color 0 0 0 0)
+  )
   (junction (at 125.73 49.53) (diameter 0) (color 0 0 0 0)
   )
@@
   )
   (junction (at 144.78 54.61) (diameter 0) (color 0 0 0 0)
+  )
+  (junction (at 125.73 157.48) (diameter 0) (color 0 0 0 0)
   )
   (no_connect (at 193.04 44.45))
@@
     (stroke (width 0) (type default))
   )
+  (wire (pts (xy 141.605 64.77) (xy 133.35 64.77))
+    (stroke (width 0) (type default))
+  )
   (wire (pts (xy 144.78 152.4) (xy 133.35 152.4))
     (stroke (width 0) (type default))
@@
     (stroke (width 0) (type default))
   )
+  (wire (pts (xy 141.605 162.56) (xy 133.35 162.56))
+    (stroke (width 0) (type default))
+  )
   (wire (pts (xy 191.77 39.37) (xy 179.07 39.37))
     (stroke (width 0) (type default))
@@
     (stroke (width 0) (type default))
   )
+  (wire (pts (xy 141.605 114.3) (xy 133.35 114.3))
+    (stroke (width 0) (type default))
+  )
   (wire (pts (xy 152.4 119.38) (xy 158.75 119.38))
     (stroke (width 0) (type default))
+  )
+  (label "+12V_LIM" (at 141.605 162.56 180) (fields_autoplaced)
+    (effects (font (size 1.27 1.27)) (justify right bottom))
+  )
+  (label "+12V_LIM" (at 141.605 64.77 180) (fields_autoplaced)
+    (effects (font (size 1.27 1.27)) (justify right bottom))
   )
   (label "+12V_LIM" (at 189.23 39.37 180) (fields_autoplaced)
     (effects (font (size 1.27 1.27)) (justify right bottom))
   )
+  (label "+12V_LIM" (at 141.605 114.3 180) (fields_autoplaced)
+    (effects (font (size 1.27 1.27)) (justify right bottom))
+  )
   (hierarchical_label "PU_EN1" (shape input) (at 162.56 69.85 0) (fields_autoplaced)
     (effects (font (size 1.27 1.27)) (justify left))
@@
     )
   )
+  (symbol (lib_id "power:GND") (at 118.11 162.56 270) (unit 1)
+    (in_bom yes) (on_board yes) (dnp no)
+    (property "Reference" "#PWR0280" (at 111.76 162.56 0)
+      (effects (font (size 1.27 1.27)) hide)
+    )
+    (property "Value" "GND" (at 113.03 162.56 90)
+      (effects (font (size 1.27 1.27)))
+    )
+    (property "Footprint" "" (at 118.11 162.56 0)
+      (effects (font (size 1.27 1.27)) hide)
+    )
+    (property "Datasheet" "" (at 118.11 162.56 0)
+      (effects (font (size 1.27 1.27)) hide)
+    )
+    (pin "1")
+    (instances
+      (project "alphax_4ch"
+        (path "/63d2dd9f-d5ff-4811-a88d-0ba932475460"
+          (reference "#PWR0280") (unit 1)
+        )
+        (path "/63d2dd9f-d5ff-4811-a88d-0ba932475460/f47356e8-3d69-412e-a5c7-6fefd0461582"
+          (reference "#PWR067") (unit 1)
+        )
+      )
+    )
+  )
   (symbol (lib_id "hellen-one-common:MOSFET-N") (at 147.32 119.38 0) (mirror y) (unit 1)
     (in_bom yes) (on_board yes) (dnp no)
@@
     )
   )
+  (symbol (lib_id "power:GND") (at 118.11 64.77 270) (unit 1)
+    (in_bom yes) (on_board yes) (dnp no)
+    (property "Reference" "#PWR0280" (at 111.76 64.77 0)
+      (effects (font (size 1.27 1.27)) hide)
+    )
+    (property "Value" "GND" (at 113.03 64.77 90)
+      (effects (font (size 1.27 1.27)))
+    )
+    (property "Footprint" "" (at 118.11 64.77 0)
+      (effects (font (size 1.27 1.27)) hide)
+    )
+    (property "Datasheet" "" (at 118.11 64.77 0)
+      (effects (font (size 1.27 1.27)) hide)
+    )
+    (pin "1")
+    (instances
+      (project "alphax_4ch"
+        (path "/63d2dd9f-d5ff-4811-a88d-0ba932475460"
+          (reference "#PWR0280") (unit 1)
+        )
+        (path "/63d2dd9f-d5ff-4811-a88d-0ba932475460/f47356e8-3d69-412e-a5c7-6fefd0461582"
+          (reference "#PWR065") (unit 1)
+        )
+      )
+    )
+  )
   (symbol (lib_name "MOSFET-P_2") (lib_id "hellen-one-common:MOSFET-P") (at 128.27 104.14 180) (unit 1)
     (in_bom yes) (on_board yes) (dnp no)
@@
     )
   )
+  (symbol (lib_id "Diode:BAT54S") (at 125.73 162.56 0) (mirror x) (unit 1)
+    (in_bom yes) (on_board yes) (dnp no)
+    (property "Reference" "D78" (at 128.27 160.02 0)
+      (effects (font (size 1.27 1.27)))
+    )
+    (property "Value" "BAT54S" (at 129.54 165.1 0)
+      (effects (font (size 1.27 1.27)))
+    )
+    (property "Footprint" "Package_TO_SOT_SMD:SOT-23" (at 127.635 165.735 0)
+      (effects (font (size 1.27 1.27)) (justify left) hide)
+    )
+    (property "Datasheet" "https://www.diodes.com/assets/Datasheets/ds11005.pdf" (at 122.682 162.56 0)
+      (effects (font (size 1.27 1.27)) hide)
+    )
+    (property "LCSC" "C408389" (at 125.73 162.56 0)
+      (effects (font (size 1.27 1.27)) hide)
+    )
+    (pin "1")
+    (pin "2")
+    (pin "3")
+    (instances
+      (project "alphax_4ch"
+        (path "/63d2dd9f-d5ff-4811-a88d-0ba932475460"
+          (reference "D78") (unit 1)
+        )
+        (path "/63d2dd9f-d5ff-4811-a88d-0ba932475460/f47356e8-3d69-412e-a5c7-6fefd0461582"
+          (reference "D23") (unit 1)
+        )
+      )
+    )
+  )
   (symbol (lib_id "hellen-one-common:Res") (at 121.92 59.69 0) (mirror y) (unit 1)
     (in_bom yes) (on_board yes) (dnp no)
@@
         (path "/63d2dd9f-d5ff-4811-a88d-0ba932475460/f47356e8-3d69-412e-a5c7-6fefd0461582"
           (reference "R41") (unit 1)
+        )
+      )
+    )
+  )
+  (symbol (lib_id "Diode:BAT54S") (at 125.73 64.77 0) (mirror x) (unit 1)
+    (in_bom yes) (on_board yes) (dnp no)
+    (property "Reference" "D78" (at 128.27 62.23 0)
+      (effects (font (size 1.27 1.27)))
+    )
+    (property "Value" "BAT54S" (at 129.54 67.31 0)
+      (effects (font (size 1.27 1.27)))
+    )
+    (property "Footprint" "Package_TO_SOT_SMD:SOT-23" (at 127.635 67.945 0)
+      (effects (font (size 1.27 1.27)) (justify left) hide)
+    )
+    (property "Datasheet" "https://www.diodes.com/assets/Datasheets/ds11005.pdf" (at 122.682 64.77 0)
+      (effects (font (size 1.27 1.27)) hide)
+    )
+    (property "LCSC" "C408389" (at 125.73 64.77 0)
+      (effects (font (size 1.27 1.27)) hide)
+    )
+    (pin "1")
+    (pin "2")
+    (pin "3")
+    (instances
+      (project "alphax_4ch"
+        (path "/63d2dd9f-d5ff-4811-a88d-0ba932475460"
+          (reference "D78") (unit 1)
+        )
+        (path "/63d2dd9f-d5ff-4811-a88d-0ba932475460/f47356e8-3d69-412e-a5c7-6fefd0461582"
+          (reference "D18") (unit 1)
         )
       )
@@
     )
   )
+  (symbol (lib_id "power:GND") (at 118.11 114.3 270) (unit 1)
+    (in_bom yes) (on_board yes) (dnp no)
+    (property "Reference" "#PWR0280" (at 111.76 114.3 0)
+      (effects (font (size 1.27 1.27)) hide)
+    )
+    (property "Value" "GND" (at 113.03 114.3 90)
+      (effects (font (size 1.27 1.27)))
+    )
+    (property "Footprint" "" (at 118.11 114.3 0)
+      (effects (font (size 1.27 1.27)) hide)
+    )
+    (property "Datasheet" "" (at 118.11 114.3 0)
+      (effects (font (size 1.27 1.27)) hide)
+    )
+    (pin "1")
+    (instances
+      (project "alphax_4ch"
+        (path "/63d2dd9f-d5ff-4811-a88d-0ba932475460"
+          (reference "#PWR0280") (unit 1)
+        )
+        (path "/63d2dd9f-d5ff-4811-a88d-0ba932475460/f47356e8-3d69-412e-a5c7-6fefd0461582"
+          (reference "#PWR066") (unit 1)
+        )
+      )
+    )
+  )
   (symbol (lib_id "hellen-one-common:Res") (at 111.76 157.48 0) (mirror y) (unit 1)
     (in_bom yes) (on_board yes) (dnp no)
@@
         )
       )
+    )
+  )
+  (symbol (lib_id "Diode:BAT54S") (at 125.73 114.3 0) (mirror x) (unit 1)
+    (in_bom yes) (on_board yes) (dnp no)
+    (property "Reference" "D78" (at 128.27 111.76 0)
+      (effects (font (size 1.27 1.27)))
+    )
+    (property "Value" "BAT54S" (at 129.54 116.84 0)
+      (effects (font (size 1.27 1.27)))
+    )
+    (property "Footprint" "Package_TO_SOT_SMD:SOT-23" (at 127.635 117.475 0)
+      (effects (font (size 1.27 1.27)) (justify left) hide)
+    )
+    (property "Datasheet" "https://www.diodes.com/assets/Datasheets/ds11005.pdf" (at 122.682 114.3 0)
+      (effects (font (size 1.27 1.27)) hide)
+    )
+    (property "LCSC" "C408389" (at 125.73 114.3 0)
+      (effects (font (size 1.27 1.27)) hide)
+    )
+    (pin "1")
+    (pin "2")
+    (pin "3")
+    (instances
+      (project "alphax_4ch"
+        (path "/63d2dd9f-d5ff-4811-a88d-0ba932475460"
+          (reference "D78") (unit 1)
+        )
+        (path "/63d2dd9f-d5ff-4811-a88d-0ba932475460/f47356e8-3d69-412e-a5c7-6fefd0461582"
+          (reference "D19") (unit 1)
+        )
+      )

Commit message: PN fixes
Parts:
- D78: LCSC C408389 -> C47546
Changed lines of the file:
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@@
       (effects (font (size 1.27 1.27)) hide)
     )
-    (property "LCSC" "C408389" (at 125.73 162.56 0)
+    (property "LCSC" "C47546" (at 125.73 162.56 0)
       (effects (font (size 1.27 1.27)) hide)
     )
@@
       (effects (font (size 1.27 1.27)) hide)
     )
-    (property "LCSC" "C408389" (at 125.73 64.77 0)
+    (property "LCSC" "C47546" (at 125.73 64.77 0)
       (effects (font (size 1.27 1.27)) hide)
     )
@@
       (effects (font (size 1.27 1.27)) hide)
     )
-    (property "LCSC" "C408389" (at 125.73 114.3 0)
-      (effects (font (size 1.27 1.27)) hide)
-    )
+    (property "LCSC" "C47546" (at 125.73 114.3 0)
+      (effects (font (size 1.27 1.27)) hide)
+    )

Commit message: Rev H*: #140, #142, #144, #145
Parts:
- R21, R23, R34, R36, R75, R77: footprint hellen-one-common:R1206 -> Resistor_SMD:R_1206_3216Metric
Changed lines of the file:
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@@
       (effects (font (size 1.27 1.27)))
     )
-    (property "Footprint" "hellen-one-common:R1206" (at 107.95 113.03 0)
+    (property "Footprint" "Resistor_SMD:R_1206_3216Metric" (at 107.95 113.03 0)
       (effects (font (size 1.27 1.27)) hide)
     )
@@
       (effects (font (size 1.27 1.27)))
     )
-    (property "Footprint" "hellen-one-common:R1206" (at 118.11 161.29 0)
+    (property "Footprint" "Resistor_SMD:R_1206_3216Metric" (at 118.11 161.29 0)
       (effects (font (size 1.27 1.27)) hide)
     )
@@
       (effects (font (size 1.27 1.27)))
     )
-    (property "Footprint" "hellen-one-common:R1206" (at 118.11 63.5 0)
+    (property "Footprint" "Resistor_SMD:R_1206_3216Metric" (at 118.11 63.5 0)
       (effects (font (size 1.27 1.27)) hide)
     )
@@
       (effects (font (size 1.27 1.27)))
     )
-    (property "Footprint" "hellen-one-common:R1206" (at 107.95 63.5 0)
+    (property "Footprint" "Resistor_SMD:R_1206_3216Metric" (at 107.95 63.5 0)
       (effects (font (size 1.27 1.27)) hide)
     )
@@
       (effects (font (size 1.27 1.27)))
     )
-    (property "Footprint" "hellen-one-common:R1206" (at 118.11 113.03 0)
+    (property "Footprint" "Resistor_SMD:R_1206_3216Metric" (at 118.11 113.03 0)
       (effects (font (size 1.27 1.27)) hide)
     )
@@
       (effects (font (size 1.27 1.27)))
     )
-    (property "Footprint" "hellen-one-common:R1206" (at 107.95 161.29 0)
-      (effects (font (size 1.27 1.27)) hide)
-    )
+    (property "Footprint" "Resistor_SMD:R_1206_3216Metric" (at 107.95 161.29 0)
+      (effects (font (size 1.27 1.27)) hide)
+    )

Commit message: Export
Parts:
- added D78 (x2): BAT54S, Package_TO_SOT_SMD:SOT-23, symbol Diode:BAT54S
- added Q15, Q25: AO3400A, hellen-one-common:SOT-23, symbol hellen-one-common:MOSFET-N
- added Q16, Q17, Q31, Q32: AO3401A, hellen-one-common:SOT-23, symbol hellen-one-common:MOSFET-P
- added R34, R36, R75, R77: 2k, Resistor_SMD:R_1206_3216Metric, symbol hellen-one-common:Res
- added R48, R74, R76 (x2), R93 (x2): 4.7k, hellen-one-common:R0603, symbol hellen-one-common:Res
Connections:
- net +12V_LIM: now also D78.2 (K), D78.2 (K), Q16.2 (D), Q31.2 (D)
- net GND: now also D78.1 (A), D78.1 (A), Q15.3 (S), Q25.3 (S), R48.1, R74.2
- new net: Q31.1 (G), Q32.1 (G), R76.1, R93.2
- new net: D78.3 (COM), Q32.2 (D), R77.1
- new net: Q31.3 (S), Q32.3 (S), R76.2
- new net: D78.3 (COM), Q17.2 (D), R36.1
- new net: R75.1, R77.2
- new net: R34.1, R36.2
- new net: Q16.1 (G), Q17.1 (G), R76.1, R93.2
- new net: Q16.3 (S), Q17.3 (S), R76.2
- new net: Q15.2 (D), R93.1
- new net: Q25.2 (D), R93.1
- new net LINE4: R34.2
- new net LINE5: R75.2
- new net PU_EN4: Q15.1 (G), R48.2
- new net PU_EN5: Q25.1 (G), R74.1
Other:
- moved on the sheet: C17, D55, Q15, Q16, Q17, Q2, Q25, Q31, Q32, Q4, Q5, R21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
