File: INJ4.kicad_sch (KiCad schematic)
At the start: 8 parts, among them Q26 VND14NV04-E, Q30 VND14NV04-E, Q6 VND14NV04-E, Q7 VND14NV04-E

Commit message: Export
Changed lines of the file:
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@@
         )
         (path "/63d2dd9f-d5ff-4811-a88d-0ba932475460/25155a6a-b730-4539-b065-c798d1d9d962"
-          (reference "#PWR093") (unit 1)
+          (reference "#PWR0151") (unit 1)
         )
       )
@@
         )
         (path "/63d2dd9f-d5ff-4811-a88d-0ba932475460/25155a6a-b730-4539-b065-c798d1d9d962"
-          (reference "#PWR091") (unit 1)
+          (reference "#PWR0143") (unit 1)
         )
       )
@@
         )
         (path "/63d2dd9f-d5ff-4811-a88d-0ba932475460/25155a6a-b730-4539-b065-c798d1d9d962"
-          (reference "#PWR088") (unit 1)
+          (reference "#PWR0147") (unit 1)
         )
       )
@@
         )
         (path "/63d2dd9f-d5ff-4811-a88d-0ba932475460/25155a6a-b730-4539-b065-c798d1d9d962"
-          (reference "#PWR092") (unit 1)
+          (reference "#PWR0149") (unit 1)
         )
       )
@@
         )
         (path "/63d2dd9f-d5ff-4811-a88d-0ba932475460/25155a6a-b730-4539-b065-c798d1d9d962"
-          (reference "#PWR087") (unit 1)
+          (reference "#PWR0148") (unit 1)
         )
       )
@@
         )
         (path "/63d2dd9f-d5ff-4811-a88d-0ba932475460/25155a6a-b730-4539-b065-c798d1d9d962"
-          (reference "#PWR086") (unit 1)
+          (reference "#PWR0146") (unit 1)
         )
       )
@@
         )
         (path "/63d2dd9f-d5ff-4811-a88d-0ba932475460/25155a6a-b730-4539-b065-c798d1d9d962"
-          (reference "#PWR094") (unit 1)
+          (reference "#PWR0144") (unit 1)
         )
       )
@@
       (effects (font (size 1.27 1.27)) hide)
     )
-    (property "Value" "GND" (at 129.54 128.27 0)
+    (property "Value" "GND" (at 132.08 128.27 0)
       (effects (font (size 1.27 1.27)))
     )
@@
         )
         (path "/63d2dd9f-d5ff-4811-a88d-0ba932475460/25155a6a-b730-4539-b065-c798d1d9d962"
-          (reference "#PWR090") (unit 1)
-        )
-      )
+          (reference "#PWR0145") (unit 1)
+        )
+      )
