File: LS4.kicad_sch (KiCad schematic)
At the start: 12 parts, among them Q26 VND14NV04-E, Q30 VND14NV04-E, Q6 VND14NV04-E, Q7 VND14NV04-E

Commit message: Export
Changed lines of the file:
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@@
         )
         (path "/63d2dd9f-d5ff-4811-a88d-0ba932475460/6c46a945-8c60-46f9-927f-d661c7787628"
-          (reference "#PWR098") (unit 1)
-        )
-        (path "/63d2dd9f-d5ff-4811-a88d-0ba932475460/379f9dcd-388e-47c8-940c-7787005440d1"
-          (reference "#PWR0132") (unit 1)
+          (reference "#PWR0158") (unit 1)
+        )
+        (path "/63d2dd9f-d5ff-4811-a88d-0ba932475460/379f9dcd-388e-47c8-940c-7787005440d1"
+          (reference "#PWR0181") (unit 1)
         )
       )
@@
       (effects (font (size 1.27 1.27)) hide)
     )
-    (property "Value" "GND" (at 139.7 163.83 0)
+    (property "Value" "GND" (at 142.24 163.83 0)
       (effects (font (size 1.27 1.27)))
     )
@@
         )
         (path "/63d2dd9f-d5ff-4811-a88d-0ba932475460/6c46a945-8c60-46f9-927f-d661c7787628"
-          (reference "#PWR099") (unit 1)
-        )
-        (path "/63d2dd9f-d5ff-4811-a88d-0ba932475460/379f9dcd-388e-47c8-940c-7787005440d1"
-          (reference "#PWR0134") (unit 1)
+          (reference "#PWR0159") (unit 1)
+        )
+        (path "/63d2dd9f-d5ff-4811-a88d-0ba932475460/379f9dcd-388e-47c8-940c-7787005440d1"
+          (reference "#PWR0182") (unit 1)
         )
       )
@@
         )
         (path "/63d2dd9f-d5ff-4811-a88d-0ba932475460/6c46a945-8c60-46f9-927f-d661c7787628"
-          (reference "#PWR096") (unit 1)
-        )
-        (path "/63d2dd9f-d5ff-4811-a88d-0ba932475460/379f9dcd-388e-47c8-940c-7787005440d1"
-          (reference "#PWR0131") (unit 1)
+          (reference "#PWR0154") (unit 1)
+        )
+        (path "/63d2dd9f-d5ff-4811-a88d-0ba932475460/379f9dcd-388e-47c8-940c-7787005440d1"
+          (reference "#PWR0177") (unit 1)
         )
       )
@@
         )
         (path "/63d2dd9f-d5ff-4811-a88d-0ba932475460/6c46a945-8c60-46f9-927f-d661c7787628"
-          (reference "#PWR095") (unit 1)
-        )
-        (path "/63d2dd9f-d5ff-4811-a88d-0ba932475460/379f9dcd-388e-47c8-940c-7787005440d1"
-          (reference "#PWR0130") (unit 1)
+          (reference "#PWR0153") (unit 1)
+        )
+        (path "/63d2dd9f-d5ff-4811-a88d-0ba932475460/379f9dcd-388e-47c8-940c-7787005440d1"
+          (reference "#PWR0176") (unit 1)
         )
       )
@@
         )
         (path "/63d2dd9f-d5ff-4811-a88d-0ba932475460/6c46a945-8c60-46f9-927f-d661c7787628"
-          (reference "#PWR0101") (unit 1)
-        )
-        (path "/63d2dd9f-d5ff-4811-a88d-0ba932475460/379f9dcd-388e-47c8-940c-7787005440d1"
-          (reference "#PWR0136") (unit 1)
+          (reference "#PWR0155") (unit 1)
+        )
+        (path "/63d2dd9f-d5ff-4811-a88d-0ba932475460/379f9dcd-388e-47c8-940c-7787005440d1"
+          (reference "#PWR0178") (unit 1)
         )
       )
@@
         )
         (path "/63d2dd9f-d5ff-4811-a88d-0ba932475460/6c46a945-8c60-46f9-927f-d661c7787628"
-          (reference "#PWR0104") (unit 1)
-        )
-        (path "/63d2dd9f-d5ff-4811-a88d-0ba932475460/379f9dcd-388e-47c8-940c-7787005440d1"
-          (reference "#PWR0138") (unit 1)
+          (reference "#PWR0157") (unit 1)
+        )
+        (path "/63d2dd9f-d5ff-4811-a88d-0ba932475460/379f9dcd-388e-47c8-940c-7787005440d1"
+          (reference "#PWR0180") (unit 1)
         )
       )
@@
         )
         (path "/63d2dd9f-d5ff-4811-a88d-0ba932475460/6c46a945-8c60-46f9-927f-d661c7787628"
-          (reference "#PWR0100") (unit 1)
-        )
-        (path "/63d2dd9f-d5ff-4811-a88d-0ba932475460/379f9dcd-388e-47c8-940c-7787005440d1"
-          (reference "#PWR0135") (unit 1)
+          (reference "#PWR0152") (unit 1)
+        )
+        (path "/63d2dd9f-d5ff-4811-a88d-0ba932475460/379f9dcd-388e-47c8-940c-7787005440d1"
+          (reference "#PWR0175") (unit 1)
         )
       )
@@
         )
         (path "/63d2dd9f-d5ff-4811-a88d-0ba932475460/6c46a945-8c60-46f9-927f-d661c7787628"
-          (reference "#PWR0103") (unit 1)
-        )
-        (path "/63d2dd9f-d5ff-4811-a88d-0ba932475460/379f9dcd-388e-47c8-940c-7787005440d1"
-          (reference "#PWR0137") (unit 1)
-        )
-      )
+          (reference "#PWR0156") (unit 1)
+        )
+        (path "/63d2dd9f-d5ff-4811-a88d-0ba932475460/379f9dcd-388e-47c8-940c-7787005440d1"
+          (reference "#PWR0179") (unit 1)
+        )
+      )
