File: MAP.kicad_sch (KiCad schematic)
At the start: 2 parts, among them U3 MPXH6400A

Commit message: Export
Parts:
- removed U3: MPXH6400A, hellen-one-common:MPXH6400A-SSOP8, symbol MPX-4_MAP:MPX4_MAP
- added U3: MPXH6400A, hellen-one-common:MPXH6400A-SSOP8, symbol hellen-one-common:MPX4_MAP
Connections:
- net +5VA: now also U3.2 (Vs)
- net GND: now also U3.3 (GND)
- net OUT: now also U3.4 (Vout)
Changed lines of the file:
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@@
       (effects (font (size 1.27 1.27)) hide)
     )
-    (property "Value" "GND" (at 159.385 86.36 90)
+    (property "Value" "GND" (at 158.75 86.36 90)
       (effects (font (size 1.27 1.27)))
     )
@@
         )
         (path "/63d2dd9f-d5ff-4811-a88d-0ba932475460/aafb5e2e-7f5c-429b-85e5-76b90069790c"
-          (reference "#PWR0149") (unit 1)
-        )
-      )
-    )
-  )
-  (symbol (lib_id "MPX-4_MAP:MPX4_MAP") (at 146.05 85.09 180) (unit 1)
-    (in_bom yes) (on_board yes) (dnp no)
-    (property "Reference" "U3" (at 142.24 78.74 0)
-      (effects (font (size 1.524 1.524)) (justify left))
-    )
-    (property "Value" "MPXH6400A" (at 149.86 81.28 0)
-      (effects (font (size 1.524 1.524)) (justify left))
-    )
-    (property "Footprint" "hellen-one-common:MPXH6400A-SSOP8" (at 146.05 85.09 0)
-      (effects (font (size 1.27 1.27)) hide)
-    )
-    (property "Datasheet" "" (at 146.05 85.09 0)
-      (effects (font (size 1.524 1.524)) hide)
-    )
-    (property "LCSC" "C511770" (at 146.05 85.09 0)
-      (effects (font (size 1.27 1.27)) hide)
-    )
-    (pin "1")
-    (pin "2")
-    (pin "3")
-    (pin "4")
-    (pin "5")
-    (pin "6")
-    (pin "7")
-    (pin "8")
-    (instances
-      (project "alphax_4ch"
-        (path "/63d2dd9f-d5ff-4811-a88d-0ba932475460"
-          (reference "U3") (unit 1)
-        )
-        (path "/63d2dd9f-d5ff-4811-a88d-0ba932475460/aafb5e2e-7f5c-429b-85e5-76b90069790c"
-          (reference "U3") (unit 1)
+          (reference "#PWR0202") (unit 1)
         )
       )
@@
       (effects (font (size 1.27 1.27)) hide)
     )
-    (property "Value" "GND" (at 165.1 100.965 0)
+    (property "Value" "GND" (at 165.1 100.33 0)
       (effects (font (size 1.27 1.27)))
     )
@@
         )
         (path "/63d2dd9f-d5ff-4811-a88d-0ba932475460/aafb5e2e-7f5c-429b-85e5-76b90069790c"
-          (reference "#PWR0151") (unit 1)
+          (reference "#PWR0201") (unit 1)
         )
       )
@@
         )
       )
+    )
+  )
+  (symbol (lib_id "hellen-one-common:MPX4_MAP") (at 146.05 85.09 180) (unit 1)
+    (in_bom yes) (on_board yes) (dnp no) (fields_autoplaced)
+    (property "Reference" "U3" (at 142.24 77.47 0)
+      (effects (font (size 1.524 1.524)))
+    )
+    (property "Value" "MPXH6400A" (at 142.24 80.01 0)
+      (effects (font (size 1.524 1.524)))
+    )
+    (property "Footprint" "hellen-one-common:MPXH6400A-SSOP8" (at 146.05 85.09 0)
+      (effects (font (size 1.27 1.27)) hide)
+    )
+    (property "Datasheet" "" (at 146.05 85.09 0)
+      (effects (font (size 1.524 1.524)) hide)
+    )
+    (property "LCSC" "C511770" (at 146.05 85.09 0)
+      (effects (font (size 1.27 1.27)) hide)
+    )
+    (pin "1")
+    (pin "2")
+    (pin "3")
+    (pin "4")
+    (pin "5")
+    (pin "6")
+    (pin "7")
+    (pin "8")
+    (instances
+      (project "alphax_4ch"
+        (path "/63d2dd9f-d5ff-4811-a88d-0ba932475460/aafb5e2e-7f5c-429b-85e5-76b90069790c"
+          (reference "U3") (unit 1)
+        )
+      )
