File: TACH_PU.kicad_sch (KiCad schematic)
At the start: 11 parts, among them Q1 AO3400A, Q3 AO3401A

Commit message: Fab preview
Connections:
- net +5V renamed +5VA
Changed lines of the file:
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@@
     )
   )
-  (symbol (lib_id "power:+5V") (at 88.9 40.64 0) (unit 1)
+  (symbol (lib_id "power:+5VA") (at 88.9 40.64 0) (mirror y) (unit 1)
     (in_bom yes) (on_board yes) (dnp no)
-    (property "Reference" "#PWR050" (at 88.9 44.45 0)
+    (property "Reference" "#PWR067" (at 88.9 44.45 0)
       (effects (font (size 1.27 1.27)) hide)
     )
-    (property "Value" "+5V" (at 88.9 36.83 0)
+    (property "Value" "+5VA" (at 88.9 36.83 0)
       (effects (font (size 1.27 1.27)))
     )
@@
       (project "alphax_4ch"
         (path "/63d2dd9f-d5ff-4811-a88d-0ba932475460"
-          (reference "#PWR050") (unit 1)
+          (reference "#PWR067") (unit 1)
+        )
+        (path "/63d2dd9f-d5ff-4811-a88d-0ba932475460/c3470145-cca5-462e-8136-3f6ead667763"
+          (reference "#PWR055") (unit 1)
         )
         (path "/63d2dd9f-d5ff-4811-a88d-0ba932475460/15162d4d-e221-4df0-bbe4-06499b4ace57"
-          (reference "#PWR0162") (unit 1)
+          (reference "#PWR049") (unit 1)
         )
       )

Commit message: Export
Changed lines of the file:
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@@
       (effects (font (size 1.27 1.27)) hide)
     )
-    (property "Value" "GND" (at 123.1392 80.1434 0)
+    (property "Value" "GND" (at 123.19 80.01 0)
       (effects (font (size 1.27 1.27)))
     )
@@
         )
         (path "/63d2dd9f-d5ff-4811-a88d-0ba932475460/15162d4d-e221-4df0-bbe4-06499b4ace57"
-          (reference "#PWR0164") (unit 1)
+          (reference "#PWR0215") (unit 1)
         )
       )
@@
       (effects (font (size 1.27 1.27)) hide)
     )
-    (property "Value" "GND" (at 157.48 46.736 0)
+    (property "Value" "GND" (at 157.48 46.99 0)
       (effects (font (size 1.27 1.27)))
     )
@@
         )
         (path "/63d2dd9f-d5ff-4811-a88d-0ba932475460/15162d4d-e221-4df0-bbe4-06499b4ace57"
-          (reference "#PWR0166") (unit 1)
+          (reference "#PWR0213") (unit 1)
         )
       )
@@
       (effects (font (size 1.27 1.27)) hide)
     )
-    (property "Value" "GND" (at 115.5192 73.7934 0)
+    (property "Value" "GND" (at 115.57 73.66 0)
       (effects (font (size 1.27 1.27)))
     )
@@
         )
         (path "/63d2dd9f-d5ff-4811-a88d-0ba932475460/15162d4d-e221-4df0-bbe4-06499b4ace57"
-          (reference "#PWR0163") (unit 1)
+          (reference "#PWR0216") (unit 1)
         )
       )
@@
         )
         (path "/63d2dd9f-d5ff-4811-a88d-0ba932475460/15162d4d-e221-4df0-bbe4-06499b4ace57"
-          (reference "#PWR0165") (unit 1)
-        )
-      )
+          (reference "#PWR0214") (unit 1)
+        )
+      )
